File: PCD_PLV005_Beyla/PCB_PLV005_Beyla.kicad_pcb (KiCad board)
At the start: 2 copper layers, 42 parts, among them J1 PWR/QB, J2 Switch_In, Q1 DMG2302UK-7, Q2 DMP2123L-7, U2 74HC266, U3 74HC08, U4 74HC21, U5 74LVC1G17, U6 LTC6993xS6-1

Commit message: Beyla PCB for review
Parts:
- turned C2 to 180 degrees
- turned C3 to 180 degrees
- turned C4 to 180 degrees
- turned C6 to 180 degrees
- turned D1 to 180 degrees
- turned R5 to 180 degrees
- turned R6 to 180 degrees
- turned R7 to 180 degrees
- turned R8 to 180 degrees
Routing:
- net GND: track 0.00 -> 172.4 mm, vias 0 -> 10
- net +5V: track 0.00 -> 171.2 mm, vias 0 -> 9
- net Net-(C8-Pad1): track 0.00 -> 76.2 mm, vias 0 -> 1
- net /AvionicsHeartbeatTemplate/HEARTBEAT: track 0.00 -> 71.6 mm, vias 0 -> 2
- net Net-(R4-Pad2): track 0.00 -> 68.6 mm, vias 0 -> 4
- net Net-(U3-Pad6): track 0.00 -> 43.5 mm, vias 0 -> 2
- net Net-(U3-Pad5): track 0.00 -> 39.2 mm, vias 0 -> 2
- net /AvionicsHeartbeatTemplate/HEARTBEAT_INPUT_1: track 0.00 -> 37.7 mm, vias 0 -> 2
- net Net-(Q1-Pad1): track 0.00 -> 34.6 mm, vias 0 -> 2
- net Net-(U2-Pad10): track 0.00 -> 34.6 mm, vias 0 -> 4
- net Net-(U2-Pad11): track 0.00 -> 26.5 mm, vias 0 -> 4
- net Net-(R3-Pad2): track 0.00 -> 26.3 mm, vias 0 -> 2
- net /AvionicsHeartbeatTemplate/HEARTBEAT_ADDRESS_2: track 0.00 -> 21.3 mm, vias 0 -> 2
- net /AvionicsHeartbeatTemplate/HEARTBEAT_ADDRESS_4: track 0.00 -> 19.6 mm, vias 0 -> 1
- net /AvionicsHeartbeatTemplate/HEARTBEAT_ADDRESS_3: track 0.00 -> 18.6 mm, vias 0 -> 1
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