File: PCD_PLV005_Beyla/AvionicsHeartbeat.sch (KiCad schematic (older format))
At the start: 30 parts, among them Q1 DMG2302UK-7, Q2 DMP2123L-7, U2 74HC266, U3 74HC08, U4 74HC21, U5 74LVC1G17, U6 LTC6993xS6-1

Commit message: Some Beyla Routing Changes
- Q1 and U8 overlap fixed
- Decoupling capacitors moved
- Transistor symbol fix in QB template schematic
Parts:
- Q1: symbol TemplateProject-rescue:Q_NMOS_GDS-Device -> Device:Q_NMOS_GSD
- Q2: symbol TemplateProject-rescue:Q_PMOS_GDS-Device -> Device:Q_PMOS_GSD
Changed lines of the file:
@@
 $EndComp
 $Comp
-L TemplateProject-rescue:Q_NMOS_GDS-Device Q1
+L Device:Q_NMOS_GSD Q1
 U 1 1 5FA03BC6
 P 6800 3350
@@
 $EndComp
 $Comp
-L TemplateProject-rescue:Q_PMOS_GDS-Device Q2
+L Device:Q_PMOS_GSD Q2
 U 1 1 5F9F8BCA
 P 7450 3100

Commit message: Beyla Layout Fixes
Fixed the problems with the first layout.
Parts:
- Q1: symbol Device:Q_NMOS_GSD -> PCB_PLV005_Beyla-rescue:Q_NMOS_GSD-Device
- Q2: symbol Device:Q_PMOS_GSD -> PCB_PLV005_Beyla-rescue:Q_PMOS_GSD-Device
Changed lines of the file:
@@
 $EndComp
 $Comp
-L Device:Q_NMOS_GSD Q1
+L PCB_PLV005_Beyla-rescue:Q_NMOS_GSD-Device Q1
 U 1 1 5FA03BC6
 P 6800 3350
@@
 $EndComp
 $Comp
-L Device:Q_PMOS_GSD Q2
+L PCB_PLV005_Beyla-rescue:Q_PMOS_GSD-Device Q2
 U 1 1 5F9F8BCA
 P 7450 3100
