File: PCD_PLV005_Beyla/PCB_PLV005_Beyla.sch (KiCad schematic (older format))
At the start: 8 parts, among them J1 PWR/QB, J2 Switch_In

Commit message: Beyla Layout Fixes
Fixed the problems with the first layout.
Parts:
- C8, C9: symbol Device:C -> PCB_PLV005_Beyla-rescue:C-Device
- D1: symbol Device:LED -> PCB_PLV005_Beyla-rescue:LED-Device
- J1: symbol Connector_Generic:Conn_01x08 -> PCB_PLV005_Beyla-rescue:Conn_01x08-Connector_Generic
- J2: symbol Connector_Generic:Conn_01x04 -> PCB_PLV005_Beyla-rescue:Conn_01x04-Connector_Generic
- R18, R19: symbol Device:R_US -> PCB_PLV005_Beyla-rescue:R_US-Device
- VR1: symbol boringlib:Recom_R-78c-1.0 -> PCB_PLV005_Beyla-rescue:Recom_R-78c-1.0-boringlib
Changed lines of the file:
@@
 $EndSheet
 $Comp
-L power:GND #PWR0101
+L PCB_PLV005_Beyla-rescue:GND-power #PWR0101
 U 1 1 5FB8B7CA
 P 7100 3450
@@
 	2800 4150 2650 4150
 $Comp
-L power:GND #PWR0102
+L PCB_PLV005_Beyla-rescue:GND-power #PWR0102
 U 1 1 5FB9ACDA
 P 2800 3600
@@
 	6250 3000 5800 3000
 $Comp
-L Device:C C8
+L PCB_PLV005_Beyla-rescue:C-Device C8
 U 1 1 5FBF38DA
 P 5800 3300
@@
 $EndComp
 $Comp
-L Device:C C9
+L PCB_PLV005_Beyla-rescue:C-Device C9
 U 1 1 5FBF4C36
 P 4550 3300
@@
 Connection ~ 5200 3600
 $Comp
-L power:+5V #PWR0103
+L PCB_PLV005_Beyla-rescue:+5V-power #PWR0103
 U 1 1 5FBFDEDC
 P 4550 2950
@@
 Connection ~ 4550 3000
 $Comp
-L Device:LED D1
+L PCB_PLV005_Beyla-rescue:LED-Device D1
 U 1 1 5FBFEF04
 P 4050 3000
@@
 $EndComp
 $Comp
-L Device:R_US R18
+L PCB_PLV005_Beyla-rescue:R_US-Device R18
 U 1 1 5FC06267
 P 3550 3300
@@
 	4550 2950 4550 3000
 $Comp
-L Connector_Generic:Conn_01x08 J1
+L PCB_PLV005_Beyla-rescue:Conn_01x08-Connector_Generic J1
 U 1 1 5FC2996A
 P 7300 4250
@@
 $EndComp
 $Comp
-L Connector_Generic:Conn_01x04 J2
+L PCB_PLV005_Beyla-rescue:Conn_01x04-Connector_Generic J2
 U 1 1 5FC2E912
 P 2450 4350
@@
 $EndComp
 $Comp
-L Device:R_US R19
+L PCB_PLV005_Beyla-rescue:R_US-Device R19
 U 1 1 5FC33E92
 P 2800 3850
@@
 	2650 4350 2800 4350
 $Comp
-L boringlib:Recom_R-78c-1.0 VR1
+L PCB_PLV005_Beyla-rescue:Recom_R-78c-1.0-boringlib VR1
 U 1 1 5FC3D4E7
 P 5200 3000
@@
 $EndComp
 $Comp
-L power:+5V #PWR0104
+L PCB_PLV005_Beyla-rescue:+5V-power #PWR0104
 U 1 1 5FDAF5EF
 P 2800 4500
