File: PCB_PLV001_Odin/PCB_PLV001_Odin.sch (KiCad schematic (older format))
At the start: 44 parts, among them J1 PWR/CAN/QB, J4 ROT1, J5 ROT2, U10 SN65HVD232, U7 R-78B12-2.0

Commit message: Odin routing
Connections:
- net +3V3: no longer C3.1, C4.1
- net +5V: now also C3.1, C4.1
Changed lines of the file:
@@
 Wire Wire Line
 	9550 3850 9550 3900
-$Comp
-L power:+3.3V #PWR0145
-U 1 1 5FD45242
-P 9550 3500
-AR Path="/5FD45242" Ref="#PWR0145"  Part="1"
-AR Path="/5FB797DD/5FD45242" Ref="#PWR?"  Part="1"
-F 0 "#PWR0145" H 9550 3350 50  0001 C CNN
-F 1 "+3.3V" H 9565 3673 50  0000 C CNN
-F 2 "" H 9550 3500 50  0001 C CNN
-F 3 "" H 9550 3500 50  0001 C CNN
-	1    9550 3500
-	1    0    0    -1
-$EndComp
 Wire Wire Line
 	9550 3500 9550 3550
@@
 Wire Wire Line
 	9550 2850 9550 2900
-$Comp
-L power:+3.3V #PWR0147
-U 1 1 5FD54BE6
-P 9550 2500
-AR Path="/5FD54BE6" Ref="#PWR0147"  Part="1"
-AR Path="/5FB797DD/5FD54BE6" Ref="#PWR?"  Part="1"
-F 0 "#PWR0147" H 9550 2350 50  0001 C CNN
-F 1 "+3.3V" H 9565 2673 50  0000 C CNN
-F 2 "" H 9550 2500 50  0001 C CNN
-F 3 "" H 9550 2500 50  0001 C CNN
-	1    9550 2500
-	1    0    0    -1
-$EndComp
 Wire Wire Line
 	9550 2500 9550 2550
@@
 Text Notes 1750 2000 0    50   ~ 0
 NOTE: Give this diode a big pad for heat
+$Comp
+L power:+5V #PWR?
+U 1 1 5FFCFA00
+P 9550 2500
+F 0 "#PWR?" H 9550 2350 50  0001 C CNN
+F 1 "+5V" H 9565 2673 50  0000 C CNN
+F 2 "" H 9550 2500 50  0001 C CNN
+F 3 "" H 9550 2500 50  0001 C CNN
+	1    9550 2500
+	1    0    0    -1
+$EndComp
+$Comp
+L power:+5V #PWR?
+U 1 1 5FFD04A9
+P 9550 3500
+F 0 "#PWR?" H 9550 3350 50  0001 C CNN
+F 1 "+5V" H 9565 3673 50  0000 C CNN
+F 2 "" H 9550 3500 50  0001 C CNN
+F 3 "" H 9550 3500 50  0001 C CNN
+	1    9550 3500
+	1    0    0    -1
+$EndComp
 $EndSCHEMATC
