File: PCB_PLV001_Odin/AvionicsHeartbeat.sch (KiCad schematic (older format))
At the start: 33 parts, among them Q1 DMG2302UK-7, Q2 DMP2123L-7, U1 74HC21, U2 74HC266, U3 74HC08, U4 74HC21, U5 74LVC1G17, U6 LTC6993xS6-1

Commit message: Fix transistors in heartbeat circuits
Parts:
- D2: value GREEN -> QB_IN
- D3: value BLUE -> QB_OUT
- Q1: symbol Device:Q_NMOS_GDS -> Device:Q_NMOS_GSD
Changed lines of the file:
@@
 P 8850 3500
 F 0 "D3" V 8889 3383 50  0000 R CNN
-F 1 "BLUE" V 8798 3383 50  0000 R CNN
+F 1 "QB_OUT" V 8798 3383 50  0000 R CNN
 F 2 "LED_SMD:LED_0805_2012Metric_Pad1.15x1.40mm_HandSolder" H 8850 3500 50  0001 C CNN
 F 3 "https://www.we-online.de/katalog/datasheet/150080BS75000.pdf" H 8850 3500 50  0001 C CNN
@@
 P 4250 3450
 F 0 "D2" V 4289 3332 50  0000 R CNN
-F 1 "GREEN" V 4198 3332 50  0000 R CNN
+F 1 "QB_IN" V 4198 3332 50  0000 R CNN
 F 2 "LED_SMD:LED_0805_2012Metric_Pad1.15x1.40mm_HandSolder" H 4250 3450 50  0001 C CNN
 F 3 "https://www.we-online.de/katalog/datasheet/150080GS75000.pdf" H 4250 3450 50  0001 C CNN
@@
 	6900 3100 6900 3150
 $Comp
-L Device:Q_NMOS_GDS Q1
+L Device:Q_NMOS_GSD Q1
 U 1 1 5FA03BC6
 P 6800 3350
