File: TemplateProject/AvionicsHeartbeat.sch (KiCad schematic (older format))
At the start: 33 parts, among them Q1 DMG2302UK-7, Q2 DMP2123L-7, U1 74HC21, U2 74HC266, U3 74HC08, U4 74HC21, U5 74LVC1G17, U6 LTC6993xS6-1

Commit message: Fix transistors in heartbeat circuits
Parts:
- Q1: symbol Device:Q_NMOS_GDS -> Device:Q_NMOS_GSD
- Q2: symbol Device:Q_PMOS_GDS -> Device:Q_PMOS_GSD
Changed lines of the file:
@@
 EESchema Schematic File Version 4
-LIBS:TemplateProject-cache
 EELAYER 29 0
 EELAYER END
 $Descr A4 11693 8268
 encoding utf-8
-Sheet 2 2
+Sheet 1 1
 Title ""
 Date ""
@@
 $EndComp
 $Comp
-L Device:Q_NMOS_GDS Q1
+L Device:Q_NMOS_GSD Q1
 U 1 1 5FA03BC6
 P 6800 3350
@@
 $EndComp
 $Comp
-L Device:Q_PMOS_GDS Q2
+L Device:Q_PMOS_GSD Q2
 U 1 1 5F9F8BCA
 P 7450 3100
