File: PCB_PLV007_Yggdrasil/AvionicsHeartbeat.sch (KiCad schematic (older format))
At the start: 33 parts, among them Q1 DMG2302UK-7, Q2 DMP2123L-7, U1 74HC21, U2 74HC266, U3 74HC08, U4 74HC21, U5 74LVC1G17, U6 LTC6993xS6-1

Commit message: Fix transistors in heartbeat circuits
Parts:
- removed C1, C2, C3, C4, C5, C6: 0.1uF, Capacitor_SMD:C_0603_1608Metric_Pad1.05x0.95mm_HandSolder, symbol Device:C
- removed C7: 1uF, symbol Device:C
- removed R12, R14: 47K, symbol Device:R_US
- removed R16: 1K, symbol Device:R_US
- removed unit 1 of U1
- removed unit 2 of U1
- removed unit 1 of U2
- removed unit 2 of U2
- removed unit 3 of U2
- removed unit 4 of U2
- added C? (x6): 0.1uF, Capacitor_SMD:C_0603_1608Metric_Pad1.05x0.95mm_HandSolder, symbol Device:C
- added C?: 1uF, Capacitor_SMD:C_0603_1608Metric_Pad1.05x0.95mm_HandSolder, symbol Device:C
- added R? (x2): 47K, Resistor_SMD:R_0603_1608Metric_Pad1.05x0.95mm_HandSolder, symbol Device:R_US
- added R?: 1K, Resistor_SMD:R_0603_1608Metric_Pad1.05x0.95mm_HandSolder, symbol Device:R_US
- added U? (x2): 74HC21, Package_SO:SOIC-14_3.9x8.7mm_P1.27mm, symbol boringlib:74HC21
- added U? (x4): 74HC266, Package_SO:SOIC-14_3.9x8.7mm_P1.27mm, symbol boringlib:74HC266
- D2: value GREEN -> QB_IN; Digikey 732-4983-1-ND -> (none); MFPN (none) -> 150080GS75000
- D3: value BLUE -> QB_OUT; Digikey 732-4982-1-ND -> (none); MFPN (none) -> 150080BS75000
- Q1: symbol Device:Q_NMOS_GDS -> Device:Q_NMOS_GSD; Digikey DMG2302UK-7DICT-ND -> (none); MFPN (none) -> DMG2302UK-7
- Q2: symbol Device:Q_PMOS_GDS -> Device:Q_PMOS_GSD; Digikey DMP2123LDICT-ND -> (none); MFPN (none) -> DMP2123L-7
- R10: footprint (none) -> Resistor_SMD:R_0603_1608Metric_Pad1.05x0.95mm_HandSolder; MFPN (none) -> RMCF0603FT280K
- R11: footprint (none) -> Resistor_SMD:R_0603_1608Metric_Pad1.05x0.95mm_HandSolder; MFPN (none) -> RMCF0603FT604K
- R15: footprint (none) -> Resistor_SMD:R_0603_1608Metric_Pad1.05x0.95mm_HandSolder; MFPN (none) -> RMCF0603FT47K0
- R17: footprint (none) -> Resistor_SMD:R_0603_1608Metric_Pad1.05x0.95mm_HandSolder; MFPN (none) -> RMCF0603FT1K00
- R9: footprint (none) -> Resistor_SMD:R_0603_1608Metric_Pad1.05x0.95mm_HandSolder; MFPN (none) -> RMCF0603FT1M00
- U1, U4: Digikey 296-31574-1-ND -> (none); MFPN (none) -> CD74HC21M96
- U2: Digikey 296-31804-1-ND -> (none); MFPN (none) -> SN74HC266DR
- U3: Digikey 296-14506-1-ND -> (none); MFPN (none) -> CD74HC08M96
- U5: Digikey 296-11933-1-ND -> (none); MFPN (none) -> SN74LVC1G17QDBVRQ1
- U5: MFPN (none) -> SN74LVC1G17QDBVRQ1
- U6: Digikey LTC6993CS6-1#TRMPBFCT-ND -> (none); MFPN (none) -> LTC6993CS6-1#TRMPBF

Commit message: Odin Silk, finish Yggdrasil component selection
Parts:
- R19: renamed from R1; footprint (none) -> Resistor_SMD:R_0603_1608Metric_Pad1.05x0.95mm_HandSolder
- R20: renamed from R2; footprint (none) -> Resistor_SMD:R_0603_1608Metric_Pad1.05x0.95mm_HandSolder
- R21: renamed from R3; footprint (none) -> Resistor_SMD:R_0603_1608Metric_Pad1.05x0.95mm_HandSolder
- R22: renamed from R4; footprint (none) -> Resistor_SMD:R_0603_1608Metric_Pad1.05x0.95mm_HandSolder
- R23: renamed from R5; footprint (none) -> Resistor_SMD:R_0603_1608Metric_Pad1.05x0.95mm_HandSolder
- R24: renamed from R6; footprint (none) -> Resistor_SMD:R_0603_1608Metric_Pad1.05x0.95mm_HandSolder
- R25: renamed from R7; footprint (none) -> Resistor_SMD:R_0603_1608Metric_Pad1.05x0.95mm_HandSolder
- R26: renamed from R8; footprint (none) -> Resistor_SMD:R_0603_1608Metric_Pad1.05x0.95mm_HandSolder
- gave numbers to parts that had none: 12
- renumbered D2 to D6, D3 to D7, R15 to R27, R9 to R29, R10 to R30, R11 to R31, R17 to R34, U1 to U3, U2 to U4, U3 to U5, U4 to U6, U5 to U7, U6 to U8

Commit message: Make Odin pass DRC, finish Yggdrasil
Parts:
- renumbered U3 to U4, U4 to U5, U5 to U6, U6 to U7, U7 to U8, U8 to U9
Changed lines of the file:
@@
 $EndDescr
 $Comp
-L boringlib:74HC21 U3
+L boringlib:74HC21 U4
 U 3 1 5F956B40
 P 900 1350
-F 0 "U3" H 1130 1396 50  0000 L CNN
+F 0 "U4" H 1130 1396 50  0000 L CNN
 F 1 "74HC21" H 1130 1305 50  0000 L CNN
 F 2 "Package_SO:SOIC-14_3.9x8.7mm_P1.27mm" H 900 1350 50  0001 C CNN
@@
 	2900 3950 2850 3950
 $Comp
-L boringlib:74HC266 U4
+L boringlib:74HC266 U5
 U 5 1 5F96A885
 P 1650 1350
-F 0 "U4" H 1880 1396 50  0000 L CNN
+F 0 "U5" H 1880 1396 50  0000 L CNN
 F 1 "74HC266" H 1880 1305 50  0000 L CNN
 F 2 "Package_SO:SOIC-14_3.9x8.7mm_P1.27mm" H 1650 1350 50  0001 C CNN
@@
 	1800 6150 3050 6150
 $Comp
-L boringlib:74HC21 U6
+L boringlib:74HC21 U7
 U 1 1 5F9A3A97
 P 4250 5100
-F 0 "U6" H 4250 5475 50  0000 C CNN
+F 0 "U7" H 4250 5475 50  0000 C CNN
 F 1 "74HC21" H 4250 5384 50  0000 C CNN
 F 2 "Package_SO:SOIC-14_3.9x8.7mm_P1.27mm" H 4250 5100 50  0001 C CNN
@@
 P 5000 3350
 AR Path="/5F98DD9A" Ref="U?"  Part="2"
-AR Path="/5F94F01A/5F98DD9A" Ref="U5"  Part="2"
-F 0 "U5" H 5000 3675 50  0000 C CNN
+AR Path="/5F94F01A/5F98DD9A" Ref="U6"  Part="2"
+F 0 "U6" H 5000 3675 50  0000 C CNN
 F 1 "74HC08" H 5000 3584 50  0000 C CNN
 F 2 "Package_SO:SOIC-14_3.9x8.7mm_P1.27mm" H 5000 3450 50  0001 C CNN
@@
 P 2450 1350
 AR Path="/5F99254E" Ref="U?"  Part="5"
-AR Path="/5F94F01A/5F99254E" Ref="U5"  Part="5"
-F 0 "U5" H 2680 1396 50  0000 L CNN
+AR Path="/5F94F01A/5F99254E" Ref="U6"  Part="5"
+F 0 "U6" H 2680 1396 50  0000 L CNN
 F 1 "74HC08" H 2680 1305 50  0000 L CNN
 F 2 "Package_SO:SOIC-14_3.9x8.7mm_P1.27mm" H 2450 1450 50  0001 C CNN
@@
 6.25ms timer\nw/ 16 addresses\nthis gives 10Hz cycle
 $Comp
-L Timer:LTC6993xS6-1 U8
+L Timer:LTC6993xS6-1 U9
 U 1 1 5F9E4DE4
 P 6100 3350
-F 0 "U8" H 5850 3600 50  0000 L CNN
+F 0 "U9" H 5850 3600 50  0000 L CNN
 F 1 "LTC6993xS6-1" H 6150 3600 50  0000 L CNN
 F 2 "Package_TO_SOT_SMD:TSOT-23-6" H 6100 2950 50  0001 C CNN
@@
 	7550 3750 7550 3800
 $Comp
-L boringlib:74HC21 U6
+L boringlib:74HC21 U7
 U 3 1 5FA1BD3A
 P 3200 1350
-F 0 "U6" H 3430 1396 50  0000 L CNN
+F 0 "U7" H 3430 1396 50  0000 L CNN
 F 1 "74HC21" H 3430 1305 50  0000 L CNN
 F 2 "Package_SO:SOIC-14_3.9x8.7mm_P1.27mm" H 3200 1350 50  0001 C CNN
@@
 	7550 3350 7550 3400
 $Comp
-L boringlib:74LVC1G17 U7
+L boringlib:74LVC1G17 U8
 U 1 1 5FAAF254
 P 8500 3350
-F 0 "U7" H 8500 3667 50  0000 C CNN
+F 0 "U8" H 8500 3667 50  0000 C CNN
 F 1 "74LVC1G17" H 8500 3576 50  0000 C CNN
 F 2 "Package_TO_SOT_SMD:SOT-23-5_HandSoldering" H 8500 3350 50  0001 C CNN
@@
 HEARTBEAT_BUFF
 $Comp
-L boringlib:74LVC1G17 U7
+L boringlib:74LVC1G17 U8
 U 2 1 5FAB53A5
 P 3950 1350
-F 0 "U7" H 4180 1396 50  0000 L CNN
+F 0 "U8" H 4180 1396 50  0000 L CNN
 F 1 "74LVC1G17" H 4180 1305 50  0000 L CNN
 F 2 "Package_TO_SOT_SMD:SOT-23-5_HandSoldering" H 3950 1350 50  0001 C CNN
@@
 P 3900 3250
 AR Path="/5FC35096" Ref="U?"  Part="2"
-AR Path="/5F94F01A/5FC35096" Ref="U5"  Part="1"
-F 0 "U5" H 3900 3575 50  0000 C CNN
+AR Path="/5F94F01A/5FC35096" Ref="U6"  Part="1"
+F 0 "U6" H 3900 3575 50  0000 C CNN
 F 1 "74HC08" H 3900 3484 50  0000 C CNN
 F 2 "Package_SO:SOIC-14_3.9x8.7mm_P1.27mm" H 3900 3350 50  0001 C CNN
@@
 $EndComp
 $Comp
-L boringlib:74HC21 U3
+L boringlib:74HC21 U4
 U 1 1 5FE984B4
 P 3200 3150
-F 0 "U3" H 3100 3400 50  0000 L CNN
+F 0 "U4" H 3100 3400 50  0000 L CNN
 F 1 "74HC21" H 3050 2900 50  0000 L CNN
 F 2 "Package_SO:SOIC-14_3.9x8.7mm_P1.27mm" H 3200 3150 50  0001 C CNN
@@
 $EndComp
 $Comp
-L boringlib:74HC21 U3
+L boringlib:74HC21 U4
 U 2 1 5FE9990D
 P 3200 3800
-F 0 "U3" H 3100 4050 50  0000 L CNN
+F 0 "U4" H 3100 4050 50  0000 L CNN
 F 1 "74HC21" H 3050 3550 50  0000 L CNN
 F 2 "Package_SO:SOIC-14_3.9x8.7mm_P1.27mm" H 3200 3800 50  0001 C CNN
@@
 $EndComp
 $Comp
-L boringlib:74HC266 U4
+L boringlib:74HC266 U5
 U 4 1 5FE9B538
 P 3350 6600
-F 0 "U4" H 3250 6800 50  0000 L CNN
+F 0 "U5" H 3250 6800 50  0000 L CNN
 F 1 "74HC266" H 3200 6400 50  0000 L CNN
 F 2 "Package_SO:SOIC-14_3.9x8.7mm_P1.27mm" H 3350 6600 50  0001 C CNN
@@
 $EndComp
 $Comp
-L boringlib:74HC266 U4
+L boringlib:74HC266 U5
 U 1 1 5FE9F230
 P 3350 4950
-F 0 "U4" H 3250 5150 50  0000 L CNN
+F 0 "U5" H 3250 5150 50  0000 L CNN
 F 1 "74HC266" H 3200 4750 50  0000 L CNN
 F 2 "Package_SO:SOIC-14_3.9x8.7mm_P1.27mm" H 3350 4950 50  0001 C CNN
@@
 $EndComp
 $Comp
-L boringlib:74HC266 U4
+L boringlib:74HC266 U5
 U 2 1 5FEA124F
 P 3350 5500
-F 0 "U4" H 3250 5700 50  0000 L CNN
+F 0 "U5" H 3250 5700 50  0000 L CNN
 F 1 "74HC266" H 3200 5300 50  0000 L CNN
 F 2 "Package_SO:SOIC-14_3.9x8.7mm_P1.27mm" H 3350 5500 50  0001 C CNN
@@
 $EndComp
 $Comp
-L boringlib:74HC266 U4
+L boringlib:74HC266 U5
 U 3 1 5FEA2778
 P 3350 6050
-F 0 "U4" H 3250 6250 50  0000 L CNN
+F 0 "U5" H 3250 6250 50  0000 L CNN
 F 1 "74HC266" H 3200 5850 50  0000 L CNN
 F 2 "Package_SO:SOIC-14_3.9x8.7mm_P1.27mm" H 3350 6050 50  0001 C CNN
