File: PCB_PLV007_Yggdrasil/UHBLS.sch (KiCad schematic (older format))
At the start: 34 parts, among them J2 UMBILICAL_MASTER, J3 UMBILICAL_POWER, Q3 Q_NPN_BCE, Q4 Q_NMOS_GDS, Q5 Q_PMOS_GDS, U10 BTS50055-1TMA, U4 74HC21, U9 LM2902

Commit message: Fix transistors in heartbeat circuits
Parts:
- removed C18, C21: 0.1uF, symbol Device:C
- removed C19: 0.47uF, symbol Device:C
- removed D7: 3.3V, symbol Device:D_Zener
- removed R25: 10K, symbol Device:R_US
- added C? (x2): 0.1uF, Capacitor_SMD:C_0603_1608Metric_Pad1.05x0.95mm_HandSolder, symbol Device:C
- added C?: 0.47uF, Capacitor_SMD:C_0603_1608Metric_Pad1.05x0.95mm_HandSolder, symbol Device:C
- added D?: 3.3V, Diode_SMD:D_SOD-323, symbol Device:D_Zener
- added R?: 10K, Resistor_SMD:R_0603_1608Metric_Pad1.05x0.95mm_HandSolder, symbol Device:R_US
- C20: footprint (none) -> Capacitor_SMD:C_0603_1608Metric_Pad1.05x0.95mm_HandSolder; MFPN (none) -> CL10B474KA8VPNC
- D5: footprint (none) -> Diode_SMD:D_SOD-323; MFPN (none) -> MM3Z3V3T1G
- Q3: value Q_NPN_BCE -> MMBTA06LT1G; footprint (none) -> Package_TO_SOT_SMD:SOT-23_Handsoldering; symbol Device:Q_NPN_BCE -> Device:Q_NPN_BEC; MFPN (none) -> MMBTA06LT1G
- Q4: value Q_NMOS_GDS -> DMG2302UK-7; footprint (none) -> Package_TO_SOT_SMD:SOT-23_Handsoldering; symbol Device:Q_NMOS_GDS -> Device:Q_NMOS_GSD; MFPN (none) -> DMG2302UK-7
- R23, R36, R38: footprint (none) -> Resistor_SMD:R_0603_1608Metric_Pad1.05x0.95mm_HandSolder; MFPN (none) -> RMCF0603FT10K0
- R28, R29, R30, R31, R34: footprint (none) -> Resistor_SMD:R_0603_1608Metric_Pad1.05x0.95mm_HandSolder; MFPN (none) -> RMCF0603FT1K00
- R32, R35, R37: footprint (none) -> Resistor_SMD:R_0603_1608Metric_Pad1.05x0.95mm_HandSolder; MFPN (none) -> RMCF0603FG100K
- U4: MFPN (none) -> CD74HC21M96
- U9: footprint (none) -> Package_SO:SOIC-14_3.9x8.7mm_P1.27mm; MFPN (none) -> LM2902LVQDRQ1
Other:
- note added: "The instrumentation section here has had its functionality verified through simualtion in LTSpice."
- note removed: "The instrumentation section here has had its functionality verified through simualtion"
- moved on the sheet: C20, D4, D5, D6, F2, J2, J3, Q5, R23, R24, R27, R28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

Commit message: Odin Silk, finish Yggdrasil component selection
Parts:
- D10: renamed from D6; footprint (none) -> LED_SMD:LED_0805_2012Metric_Pad1.15x1.40mm_HandSolder; MFPN (none) -> 150080GS75000
- D8: renamed from D4; footprint (none) -> LED_SMD:LED_0805_2012Metric_Pad1.15x1.40mm_HandSolder; MFPN (none) -> 150080GS75000
- F2: footprint (none) -> BoringFootprints:BelFuse_0679H; MFPN (none) -> 0679H9150-05
- J2: footprint (none) -> Connector_Molex:Molex_Micro-Fit_3.0_43650-0200_1x02_P3.00mm_Horizontal; MFPN (none) -> 0436500200
- J3: footprint (none) -> BoringFootprints:Molex_Ultra-Fit_172310-1204_1x04; MFPN (none) -> 1723101204
- Q5: value Q_PMOS_GDS -> DMP2123L-7; footprint (none) -> Package_TO_SOT_SMD:SOT-23_Handsoldering; MFPN (none) -> DMP2123L-7
- R36: renamed from R24; footprint (none) -> Resistor_SMD:R_0603_1608Metric_Pad1.05x0.95mm_HandSolder; MFPN (none) -> RMCF0603FT43K0
- R38: renamed from R27; footprint (none) -> Resistor_SMD:R_0603_1608Metric_Pad1.05x0.95mm_HandSolder; MFPN (none) -> RMCF0603FT16K0
- R39: renamed from R?; value 260K -> 261K; footprint (none) -> Resistor_SMD:R_0603_1608Metric_Pad1.05x0.95mm_HandSolder; MFPN (none) -> RMCF0603FT261K
- R40: renamed from R?; value 95K -> 95.3K; footprint (none) -> Resistor_SMD:R_0603_1608Metric_Pad1.05x0.95mm_HandSolder; MFPN (none) -> RMCF0603FT95K3
- R46: renamed from R33; footprint (none) -> Resistor_SMD:R_0603_1608Metric_Pad1.05x0.95mm_HandSolder; MFPN (none) -> RMCF0603FT2K10
- gave numbers to parts that had none: 5
- renumbered C20 to C24, D5 to D9, R23 to R35, R28 to R41, R29 to R42, R30 to R43, R31 to R44, R32 to R45, R34 to R47, R35 to R48, R36 to R49, R37 to R50, R38 to R51, U4 to U6

Commit message: Make Odin pass DRC, finish Yggdrasil
Parts:
- renumbered U9 to U10, U10 to U11, U6 to U7
Changed lines of the file:
@@
 P 5500 4300
 AR Path="/5FC5817F" Ref="U?"  Part="1"
-AR Path="/5FC40E29/5FC5817F" Ref="U6"  Part="2"
-F 0 "U6" H 5500 4675 50  0000 C CNN
+AR Path="/5FC40E29/5FC5817F" Ref="U7"  Part="2"
+F 0 "U7" H 5500 4675 50  0000 C CNN
 F 1 "74HC21" H 5500 4584 50  0000 C CNN
 F 2 "Package_SO:SOIC-14_3.9x8.7mm_P1.27mm" H 5500 4300 50  0001 C CNN
@@
 P 7800 2000
 AR Path="/5FC58189" Ref="U?"  Part="1"
-AR Path="/5FC40E29/5FC58189" Ref="U9"  Part="1"
-F 0 "U9" H 7800 2367 50  0000 C CNN
+AR Path="/5FC40E29/5FC58189" Ref="U10"  Part="1"
+F 0 "U10" H 7800 2367 50  0000 C CNN
 F 1 "LM2902" H 7800 2250 50  0000 C CNN
 F 2 "Package_SO:SOIC-14_3.9x8.7mm_P1.27mm" H 7750 2100 50  0001 C CNN
@@
 P 6250 1600
 AR Path="/5FC581AF" Ref="U?"  Part="2"
-AR Path="/5FC40E29/5FC581AF" Ref="U9"  Part="2"
-F 0 "U9" H 6350 1450 50  0000 C CNN
+AR Path="/5FC40E29/5FC581AF" Ref="U10"  Part="2"
+F 0 "U10" H 6350 1450 50  0000 C CNN
 F 1 "LM2902" H 6250 1850 50  0000 C CNN
 F 2 "Package_SO:SOIC-14_3.9x8.7mm_P1.27mm" H 6200 1700 50  0001 C CNN
@@
 P 2500 2700
 AR Path="/5FC581D3" Ref="U?"  Part="3"
-AR Path="/5FC40E29/5FC581D3" Ref="U9"  Part="3"
-F 0 "U9" H 2500 3067 50  0000 C CNN
+AR Path="/5FC40E29/5FC581D3" Ref="U10"  Part="3"
+F 0 "U10" H 2500 3067 50  0000 C CNN
 F 1 "LM2902" H 2500 2976 50  0000 C CNN
 F 2 "Package_SO:SOIC-14_3.9x8.7mm_P1.27mm" H 2450 2800 50  0001 C CNN
@@
 P 2500 4000
 AR Path="/5FC7C182" Ref="U?"  Part="3"
-AR Path="/5FC40E29/5FC7C182" Ref="U9"  Part="4"
-F 0 "U9" H 2500 4367 50  0000 C CNN
+AR Path="/5FC40E29/5FC7C182" Ref="U10"  Part="4"
+F 0 "U10" H 2500 4367 50  0000 C CNN
 F 1 "LM2902" H 2500 4276 50  0000 C CNN
 F 2 "Package_SO:SOIC-14_3.9x8.7mm_P1.27mm" H 2450 4100 50  0001 C CNN
@@
 P 1450 5200
 AR Path="/5FC92898" Ref="U?"  Part="2"
-AR Path="/5FC40E29/5FC92898" Ref="U9"  Part="5"
-F 0 "U9" H 1550 5200 50  0000 C CNN
+AR Path="/5FC40E29/5FC92898" Ref="U10"  Part="5"
+F 0 "U10" H 1550 5200 50  0000 C CNN
 F 1 "LM2902" H 1100 5200 50  0000 C CNN
 F 2 "Package_SO:SOIC-14_3.9x8.7mm_P1.27mm" H 1400 5300 50  0001 C CNN
@@
 P 7050 1400
 AR Path="/5FC580B1" Ref="U?"  Part="1"
-AR Path="/5FC40E29/5FC580B1" Ref="U10"  Part="1"
-F 0 "U10" H 6850 1650 50  0000 C CNN
+AR Path="/5FC40E29/5FC580B1" Ref="U11"  Part="1"
+F 0 "U11" H 6850 1650 50  0000 C CNN
 F 1 "BTS50055-1TMA" H 7400 1650 50  0000 C CNN
 F 2 "Package_TO_SOT_SMD:TO-263-7_TabPin4" H 7850 1150 50  0001 C CNN
