File: PCB_PLV006_Freya/AvionicsHeartbeat.sch (KiCad schematic (older format))
At the start: 33 parts, among them Q1 DMG2302UK-7, Q2 DMP2123L-7, U1 74HC21, U2 74HC266, U3 74HC08, U4 74HC21, U5 74LVC1G17, U6 LTC6993xS6-1

Commit message: Fix library and add act
Parts:
- U3: symbol boringlib:74HC08 -> PCB_PLV006_Freya-rescue:74HC08-boringlib
Changed lines of the file:
@@
 EESchema Schematic File Version 4
 LIBS:PCB_PLV006_Freya-cache
-EELAYER 29 0
+EELAYER 30 0
 EELAYER END
 $Descr A4 11693 8268
@@
 $EndComp
 $Comp
-L boringlib:74HC08 U3
+L PCB_PLV006_Freya-rescue:74HC08-boringlib U3
 U 1 1 5F9890B3
 P 3900 3250
@@
 $EndComp
 $Comp
-L boringlib:74HC08 U3
+L PCB_PLV006_Freya-rescue:74HC08-boringlib U3
 U 2 1 5F98DD9A
 P 5000 3350
@@
 $EndComp
 $Comp
-L boringlib:74HC08 U3
+L PCB_PLV006_Freya-rescue:74HC08-boringlib U3
 U 5 1 5F99254E
 P 2450 1350

Commit message: Freya stuff
Parts:
- U1, U4: symbol boringlib:74HC21 -> PCB_PLV006_Freya-rescue:74HC21-boringlib
Changed lines of the file:
@@
 $EndDescr
 $Comp
-L boringlib:74HC21 U1
+L PCB_PLV006_Freya-rescue:74HC21-boringlib U1
 U 1 1 5F953590
 P 3200 3150
+AR Path="/5F953590" Ref="U1"  Part="1"
+AR Path="/5F94F01A/5F953590" Ref="U1"  Part="1"
 F 0 "U1" H 3200 3525 50  0000 C CNN
 F 1 "74HC21" H 3200 3434 50  0000 C CNN
@@
 $EndComp
 $Comp
-L boringlib:74HC21 U1
+L PCB_PLV006_Freya-rescue:74HC21-boringlib U1
 U 2 1 5F9550C5
 P 3200 3800
+AR Path="/5F9550C5" Ref="U1"  Part="2"
+AR Path="/5F94F01A/5F9550C5" Ref="U1"  Part="2"
 F 0 "U1" H 3200 4175 50  0000 C CNN
 F 1 "74HC21" H 3200 4084 50  0000 C CNN
@@
 $EndComp
 $Comp
-L boringlib:74HC21 U1
+L PCB_PLV006_Freya-rescue:74HC21-boringlib U1
 U 3 1 5F956B40
 P 900 1350
+AR Path="/5F956B40" Ref="U1"  Part="3"
+AR Path="/5F94F01A/5F956B40" Ref="U1"  Part="3"
 F 0 "U1" H 1130 1396 50  0000 L CNN
 F 1 "74HC21" H 1130 1305 50  0000 L CNN
@@
 	1800 6150 3050 6150
 $Comp
-L boringlib:74HC21 U4
+L PCB_PLV006_Freya-rescue:74HC21-boringlib U4
 U 1 1 5F9A3A97
 P 4250 5100
+AR Path="/5F9A3A97" Ref="U4"  Part="1"
+AR Path="/5F94F01A/5F9A3A97" Ref="U4"  Part="1"
 F 0 "U4" H 4250 5475 50  0000 C CNN
 F 1 "74HC21" H 4250 5384 50  0000 C CNN
@@
 	7550 3750 7550 3800
 $Comp
-L boringlib:74HC21 U4
+L PCB_PLV006_Freya-rescue:74HC21-boringlib U4
 U 3 1 5FA1BD3A
 P 3200 1350
+AR Path="/5FA1BD3A" Ref="U4"  Part="3"
+AR Path="/5F94F01A/5FA1BD3A" Ref="U4"  Part="3"
 F 0 "U4" H 3430 1396 50  0000 L CNN
 F 1 "74HC21" H 3430 1305 50  0000 L CNN

Commit message: Done with Freya for FDP
Parts:
- added C23, C24: 0.1uF, Capacitor_SMD:C_0603_1608Metric_Pad1.05x0.95mm_HandSolder, symbol Device:C
- added R22: 1M, Resistor_SMD:R_0603_1608Metric_Pad1.05x0.95mm_HandSolder, symbol Device:R_US
- added R23: 392K, Resistor_SMD:R_0603_1608Metric_Pad1.05x0.95mm_HandSolder, symbol Device:R_US
- added R24: 118K, Resistor_SMD:R_0603_1608Metric_Pad1.05x0.95mm_HandSolder, symbol Device:R_US
- added U14: LTC6991, Package_TO_SOT_SMD:TSOT-23-6_HandSoldering, symbol boringlib:LTC6991
- added U15: 74LV163A, Package_SO:SOIC-16_3.9x9.9mm_P1.27mm, symbol boringlib:74LV163A
- C7: footprint (none) -> Capacitor_SMD:C_0603_1608Metric_Pad1.05x0.95mm_HandSolder
- R1, R10, R11, R12, R14, R15, R16, R17, R2, R3, R4, R5, R6, R7, R8, R9: footprint (none) -> Resistor_SMD:R_0603_1608Metric_Pad1.05x0.95mm_HandSolder
Connections:
- net +5V: now also C23.1, C24.1, R22.1, U14.5 (V+), U15.1 (~CLR~), U15.10 (ENT), U15.16 (VCC), U15.7 (ENP), U15.9 (~LOAD~)
- net GND: now also C23.2, C24.2, R23.2, R24.2, U14.1 (RST), U14.2 (GND), U15.8 (GND)
- net HEARTBEAT_ADDRESS_1: now also U15.14 (QA)
- net HEARTBEAT_ADDRESS_2: now also U15.13 (QB)
- net HEARTBEAT_ADDRESS_3: now also U15.12 (QC)
- net HEARTBEAT_ADDRESS_4: now also U15.11 (QD)
- new net: R24.1, U14.3 (SET)
- new net: R22.2, R23.1, U14.4 (DIV)
- new net: U14.6 (VOUT), U15.2 (CLK)
- no-connect marks 0 -> 5
