File: PCB_PLV006_Freya/PCB_PLV006_Freya.sch (KiCad schematic (older format))
At the start: 3 parts

Commit message: Work on Freya
Parts:
- added C? (x2): C, symbol Device:C
- added C? (x2): 0.1uF, symbol Device:C
- added JP?: CAN_TERM, symbol Device:Jumper_NC_Small
- added R?: R_US, symbol Device:R_US
- added R?: 10K, symbol Device:R_US
- added U?: SN65HVD232, Package_SO:SOIC-8_3.9x4.9mm_P1.27mm, symbol Interface_CAN_LIN:SN65HVD232
- added Y?: Crystal, symbol Device:Crystal
Connections:
- net +3V3: now also C?.1, C?.1, R?.1, U?.3 (VCC)
- net GND: now also U?.9 (VSS), C?.2, C?.2, C?.2, C?.2, U?.2 (GND)
- net CAN_nCS: now reaches J?.15 (GPIO22)
- net CAN_nCS: now also U?.16 (~CS)
- net CAN_nRESET: now reaches J?.16 (GPIO23)
- net CAN_nRESET: now also U?.17 (~RESET), R?.2
- net CAN_MISO: now reaches J?.35 (GPIO19/MISO1)
- net CAN_MISO: now also U?.15 (SO)
- net CAN_MOSI: now reaches J?.38 (GPIO20/MOSI1)
- net CAN_MOSI: now also U?.14 (SI)
- net CAN_SCLK: now reaches J?.40 (GPIO21/SCLK1)
- net CAN_SCLK: now also U?.13 (SCK)
- net CAN_TX: now reaches U?.1 (TXCAN)
- net CAN_TX: now also U?.1 (D)
- net CAN_RX: now reaches U?.2 (RXCAN)
- net CAN_RX: now also U?.4 (R)
- net at U?.7 (OSC2): now also C?.1, Y?.2
- net at U?.8 (OSC1): now also C?.1, Y?.1
- new net: JP?.1, R?.1
- new net CANH: R?.2, U?.7 (CANH)
- new net CANL: JP?.2, U?.6 (CANL)
- no-connect marks 0 -> 7
Other:
- moved on the sheet: J?, U?

Commit message: Work on Freya
Parts:
- added C? (x2): 1uF, symbol Device:C
- added C? (x6): 10uF, symbol Device:C
- added C? (x3): 0.1uF, symbol Device:C
- added J?: RJ45, symbol Connector:RJ45
- added J?: POW_IN, symbol Connector_Generic:Conn_01x04
- added R?: 1M, symbol Device:R_US
- added R?: 392K, symbol Device:R_US
- added R?: 118K, symbol Device:R_US
- added U?: ISO1432BDWR, symbol boringlib:ISO1432BDWR
- added U?: AZ1117-5.0, symbol Regulator_Linear:AZ1117-5.0
- added U?: R-78B5.0-2.0, Converter_DCDC:Converter_DCDC_RECOM_R-78B-2.0_THT, symbol Regulator_Switching:R-78B5.0-2.0
- added U?: LTC6991, Package_TO_SOT_SMD:TSOT-23-6_HandSoldering, symbol boringlib:LTC6991
Connections:
- net +3V3: now also C?.1, C?.1, U?.1 (VCC1), U?.2 (VO)
- net +5V: now also C?.1, C?.1, R?.1, U?.3 (OUT), U?.3 (VI), U?.5 (V+)
- net GND: now also C?.2, C?.2, C?.2, C?.2, C?.2, C?.2, R?.2, R?.2, U?.1 (GND), U?.1 (RST), U?.2 (GND), U?.2 (GND), U?.2 (GND1), U?.8 (GND1)
- net 485_RX: now reaches J?.10 (GPIO15/RXD)
- net 485_RX: now also U?.3 (R)
- net 485_nRE: now reaches J?.18 (GPIO24)
- net 485_nRE: now also U?.4 (~RE~)
- net 485_DE: now reaches J?.22 (GPIO25)
- net 485_DE: now also U?.5 (DE)
- net 485_TX: now reaches J?.8 (GPIO14/TXD)
- net 485_TX: now also U?.6 (D)
- net +28V: now reaches U?.A1 (IN+)
- net +28V: now also C?.1, C?.1, J?.3 (Pin_3), J?.4 (Pin_4)
- net +24V: now reaches U?.A2 (OUT+)
- net +24V: now also U?.C2 (OUT+), C?.1, C?.1, C?.1, C?.1, U?.1 (IN)
- net at U?.B2 (OUT-): now also U?.D2 (OUT-), C?.2, C?.2, C?.2
- net GNDA: now reaches U?.E1 (IN-)
- net GNDA: now also C?.2, C?.2, J?.1 (Pin_1), J?.2 (Pin_2), U?.15 (GND2), U?.9 (GND2)
- new net: J?.1, U?.11 (Y)
- new net: J?.4, U?.12 (Z)
- new net: J?.5, U?.13 (B)
- new net: J?.8, U?.14 (A)
- new net: R?.1, U?.3 (SET)
- new net: R?.1, R?.2, U?.4 (DIV)
- new net +5VA: C?.1, U?.16 (VCC2)
- no-connect marks 7 -> 14
Other:
- moved on the sheet: J?, U?

Commit message: Idek anymore
Other:
- note added: "TODO:\nUHB\nQB Master counter\nOutput conns\n"
- moved on the sheet: C?, J?, R?, U?

Commit message: Freya stuff
Parts:
- added C? (x2): 0.1uF, symbol Device:C
- added U?: 74LV163A, symbol boringlib:74LV163A
Connections:
- net +5V: now also C?.1, C?.1, U?.1 (~CLR~), U?.10 (ENT), U?.16 (VCC), U?.7 (ENP), U?.9 (~LOAD~)
- net GND: now also C?.2, C?.2, U?.8 (GND)
- net at U?.6 (VOUT): now also U?.2 (CLK)
- new net HEARTBEAT_ADDRESS_1: U?.14 (QA)
- new net HEARTBEAT_ADDRESS_2: U?.13 (QB)
- new net HEARTBEAT_ADDRESS_3: U?.12 (QC)
- new net HEARTBEAT_ADDRESS_4: U?.11 (QD)
- no-connect marks 14 -> 19
Other:
- note added: "TODO:\nUHB\nOutput conns\n"
- note removed: "TODO:\nUHB\nQB Master counter\nOutput conns\n"
- moved on the sheet: R?, U?

Commit message: Done with Freya for FDP
Parts:
- removed C? (x2): 0.1uF, symbol Device:C
- removed R?: 1M, symbol Device:R_US
- removed R?: 392K, symbol Device:R_US
- removed R?: 118K, symbol Device:R_US
- removed U?: 74LV163A, symbol boringlib:74LV163A
- removed U?: LTC6991, Package_TO_SOT_SMD:TSOT-23-6_HandSoldering, symbol boringlib:LTC6991
- added D1: D_Schottky, BoringFootprints:DO-221AC, symbol Device:D_Schottky
- added J3: UHB, Connector_Molex:Molex_Micro-Fit_3.0_43045-0400_2x02_P3.00mm_Horizontal, symbol Connector_Generic:Conn_01x02
- added K1: G5Q-1A, Relay_THT:Relay_SPST_Omron-G5Q-1A, symbol Relay:G5Q-1A
- added Q3: Q_NMOS_GSD, Package_TO_SOT_SMD:SOT-23_Handsoldering, symbol Device:Q_NMOS_GSD
- added R13: 540, Resistor_SMD:R_0603_1608Metric_Pad1.05x0.95mm_HandSolder, symbol Device:R_US
- added R18, R19, R30: 10K, Resistor_SMD:R_0603_1608Metric_Pad1.05x0.95mm_HandSolder, symbol Device:R_US
- added R25, R26, R27, R28, R29: 0, Resistor_SMD:R_0603_1608Metric_Pad1.05x0.95mm_HandSolder, symbol Device:R_US
- added R31: 20K, Resistor_SMD:R_0603_1608Metric_Pad1.05x0.95mm_HandSolder, symbol Device:R_US
- added U10: LTV-817, Package_DIP:DIP-4_W7.62mm, symbol Isolator:LTV-817
- C10, C12, C15, C16, C8, C9: renamed from C?; footprint (none) -> Capacitor_SMD:C_1210_3225Metric_Pad1.42x2.65mm_HandSolder
- C11, C13, C14, C19, C20, C21, C22: renamed from C?; footprint (none) -> Capacitor_SMD:C_0603_1608Metric_Pad1.05x0.95mm_HandSolder
- C17, C18: renamed from C?; value C -> 18pF; footprint (none) -> Capacitor_SMD:C_0603_1608Metric_Pad1.05x0.95mm_HandSolder
- J1: renamed from J?; footprint (none) -> BoringFootprints:Molex_Ultra-Fit_172310-1204_1x04; MFPN (none) -> 1723161204
- J2: renamed from J?; footprint (none) -> BoringFootprints:RPI4
- J4: renamed from J?; footprint (none) -> Connector_RJ:RJ45_Amphenol_RJHSE538X
- JP1: renamed from JP?; footprint (none) -> Jumper:SolderJumper-2_P1.3mm_Open_RoundedPad1.0x1.5mm
- R20: renamed from R?; footprint (none) -> Resistor_SMD:R_0603_1608Metric_Pad1.05x0.95mm_HandSolder
- R21: renamed from R?; value R_US -> 120; footprint (none) -> Resistor_SMD:R_1210_3225Metric_Pad1.42x2.65mm_HandSolder
- U12: renamed from U?; footprint (none) -> Package_SO:SOIC-16W_7.5x10.3mm_P1.27mm
- U8: renamed from U?; footprint (none) -> Package_TO_SOT_SMD:SOT-223-3_TabPin2
- U9: renamed from U?; footprint (none) -> BoringFootprints:Vicor_DCM
- Y1: renamed from Y?; value Crystal -> 8MHz; footprint (none) -> Crystal:Crystal_SMD_HC49-SD
- gave numbers to parts that had none: 3
Connections:
- net +24V: now also D1.1 (K), K1.5
- net +5V: now also R25.1, R26.1, R27.1, R28.1, R29.1, U10.4
- net AvionicsHeartbeatTemplate/HEARTBEAT_INPUT_3: now also R25.2
- net AvionicsHeartbeatTemplate/HEARTBEAT_INPUT_4: now also R26.2
- net AvionicsHeartbeatTemplate/HEARTBEAT_INPUT_5: now also R27.2
- net AvionicsHeartbeatTemplate/HEARTBEAT_INPUT_6: now also R28.2
- net AvionicsHeartbeatTemplate/HEARTBEAT_INPUT_7: now also R29.2
- net GND: now also C14.2, C15.2, C16.2, U9.B2 (OUT-), U9.D2 (OUT-), Q3.2 (S), R18.2, R31.1; no longer C21.2
- net GNDA: now also C21.2, R13.2
- net HEARTBEAT_ADDRESS_1: now also J2.24 (~CE0~/GPIO8)
- net HEARTBEAT_ADDRESS_2: now also J2.21 (MISO0/GPIO9)
- net HEARTBEAT_ADDRESS_3: now also J2.19 (MOSI0/GPIO10)
- net HEARTBEAT_ADDRESS_4: now also J2.23 (SCLK0/GPIO11)
- net at J2.27 (ID_SD/GPIO0): now also R30.1, R31.2
- net HEARTBEAT_RESTART: now reaches J2.32 (PWM0/GPIO12)
- net HEARTBEAT_RESTART: now also R19.2
- net MCU_QB_INPUT: now reaches J2.33 (PWM1/GPIO13)
- new net: D1.2 (A), K1.1, Q3.3 (D)
- new net: J3.1 (Pin_1), K1.2, U10.1
- new net: J3.2 (Pin_2), K1.3
- new net: R13.1, U10.2
- new net QB_BUFF: Q3.1 (G), R30.2
- new net UHB_OUT: R18.1, R19.1, U10.3
- no-connect marks 19 -> 14
Other:
- note added: "Outputs"
- note removed: "TODO:\nUHB\nOutput conns\n"
- moved on the sheet: C10, C12, C13, C17, C18, C19, C20, C21, C22, C8, J2, J4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
