File: PCB_PLV002_Thor/PCB_PLV002_Thor.kicad_pcb (KiCad board)
At the start: 2 copper layers, 21 parts, among them Q1 DMG2302UK-7, Q2 DMP2123L-7, U1 74HC21, U2 74HC266, U3 74HC08, U4 74HC21, U5 74LVC1G17, U6 LTC6993xS6-1, U7 SN65HVD232

Commit message: Done
Parts:
- added C10: 1uF, Capacitor_SMD:C_0603_1608Metric_Pad1.05x0.95mm_HandSolder, B.Cu at (76.0, 93.5)
- added C11: 0.1uF, Capacitor_SMD:C_0603_1608Metric_Pad1.05x0.95mm_HandSolder, B.Cu at (94.8, 105.0)
- added C12: 0.1uF, Capacitor_SMD:C_0603_1608Metric_Pad1.05x0.95mm_HandSolder, F.Cu at (157.0, 110.0)
- added C13: 0.1uF, Capacitor_SMD:C_0603_1608Metric_Pad1.05x0.95mm_HandSolder, F.Cu at (149.2, 110.0)
- added C14: 0.1uF, Capacitor_SMD:C_0603_1608Metric_Pad1.05x0.95mm_HandSolder, F.Cu at (141.5, 110.0)
- added C15: 0.1uF, Capacitor_SMD:C_0603_1608Metric_Pad1.05x0.95mm_HandSolder, F.Cu at (133.8, 110.0)
- added C16: 0.1uF, Capacitor_SMD:C_0603_1608Metric_Pad1.05x0.95mm_HandSolder, F.Cu at (141.2, 91.2)
- added C17: 0.1uF, Capacitor_SMD:C_0603_1608Metric_Pad1.05x0.95mm_HandSolder, B.Cu at (155.8, 94.8)
- added C18: 1uF, Capacitor_SMD:C_0603_1608Metric_Pad1.05x0.95mm_HandSolder, B.Cu at (155.8, 93.0)
- added C19: 0.1uF, Capacitor_SMD:C_0603_1608Metric_Pad1.05x0.95mm_HandSolder, F.Cu at (238.8, 135.8)
- added C20: 0.1uF, Capacitor_SMD:C_0603_1608Metric_Pad1.05x0.95mm_HandSolder, F.Cu at (229.2, 135.8)
- added C21: 0.1uF, Capacitor_SMD:C_0603_1608Metric_Pad1.05x0.95mm_HandSolder, F.Cu at (219.8, 135.8)
- added C22: 0.1uF, Capacitor_SMD:C_0603_1608Metric_Pad1.05x0.95mm_HandSolder, F.Cu at (210.2, 135.8)
- added C23: 0.1uF, Capacitor_SMD:C_0603_1608Metric_Pad1.05x0.95mm_HandSolder, F.Cu at (200.8, 135.8)
- added C24: 0.1uF, Capacitor_SMD:C_0603_1608Metric_Pad1.05x0.95mm_HandSolder, F.Cu at (191.2, 135.8)
- added C25: 0.1uF, Capacitor_SMD:C_0603_1608Metric_Pad1.05x0.95mm_HandSolder, F.Cu at (181.8, 135.8)
- added C26: 0.1uF, Capacitor_SMD:C_0603_1608Metric_Pad1.05x0.95mm_HandSolder, F.Cu at (172.2, 135.8)
- added C27: 0.1uF, Capacitor_SMD:C_0603_1608Metric_Pad1.05x0.95mm_HandSolder, B.Cu at (135.2, 127.8)
- added C28: 0.1uF, Capacitor_SMD:C_0603_1608Metric_Pad1.05x0.95mm_HandSolder, F.Cu at (162.8, 135.8)
- added C29: 0.1uF, Capacitor_SMD:C_0603_1608Metric_Pad1.05x0.95mm_HandSolder, F.Cu at (153.2, 135.8)
- added C30: 0.1uF, Capacitor_SMD:C_0603_1608Metric_Pad1.05x0.95mm_HandSolder, F.Cu at (115.8, 131.0)
- added C31: 0.1uF, Capacitor_SMD:C_0603_1608Metric_Pad1.05x0.95mm_HandSolder, F.Cu at (104.5, 131.0)
- added C32: 0.1uF, Capacitor_SMD:C_0603_1608Metric_Pad1.05x0.95mm_HandSolder, F.Cu at (93.2, 131.0)
- added C33: 0.1uF, Capacitor_SMD:C_0603_1608Metric_Pad1.05x0.95mm_HandSolder, F.Cu at (82.0, 131.0)
- added C34: 1uF, Capacitor_SMD:C_0603_1608Metric_Pad1.05x0.95mm_HandSolder, F.Cu at (99.0, 124.0)
- added C35: 1uF, Capacitor_SMD:C_0603_1608Metric_Pad1.05x0.95mm_HandSolder, F.Cu at (209.5, 125.0)
- added C36: 0.1uF, Capacitor_SMD:C_0603_1608Metric_Pad1.05x0.95mm_HandSolder, F.Cu at (97.5, 124.0)
- added C37: 0.1uF, Capacitor_SMD:C_0603_1608Metric_Pad1.05x0.95mm_HandSolder, F.Cu at (208.0, 125.0)
- added C38: 0.1uF, Capacitor_SMD:C_0603_1608Metric_Pad1.05x0.95mm_HandSolder, F.Cu at (86.8, 122.5)
- added C39: 0.1uF, Capacitor_SMD:C_0603_1608Metric_Pad1.05x0.95mm_HandSolder, F.Cu at (197.5, 123.5)
- added C40: 0.1uF, Capacitor_SMD:C_0603_1608Metric_Pad1.05x0.95mm_HandSolder, B.Cu at (98.8, 68.2)
- added C41: 0.1uF, Capacitor_SMD:C_0603_1608Metric_Pad1.05x0.95mm_HandSolder, B.Cu at (122.0, 68.2)
- added C42: 1uF, Capacitor_SMD:C_0603_1608Metric_Pad1.05x0.95mm_HandSolder, B.Cu at (89.5, 68.2)
- added C43: 1uF, Capacitor_SMD:C_0603_1608Metric_Pad1.05x0.95mm_HandSolder, B.Cu at (114.2, 68.2)
- added C44: 10uF, Capacitor_SMD:C_1210_3225Metric_Pad1.42x2.65mm_HandSolder, F.Cu at (80.0, 70.5)
- added C45: 1uF, Capacitor_SMD:C_0603_1608Metric_Pad1.05x0.95mm_HandSolder, F.Cu at (80.0, 66.2)
- added C46: 1uF, Capacitor_SMD:C_0603_1608Metric_Pad1.05x0.95mm_HandSolder, F.Cu at (80.0, 68.0)
- added C47: 0.1uF, Capacitor_SMD:C_0603_1608Metric_Pad1.05x0.95mm_HandSolder, F.Cu at (80.0, 64.5)
- added C48: 0.1uF, Capacitor_SMD:C_0603_1608Metric_Pad1.05x0.95mm_HandSolder, B.Cu at (146.5, 68.2)
- added C49: 0.1uF, Capacitor_SMD:C_0603_1608Metric_Pad1.05x0.95mm_HandSolder, B.Cu at (171.0, 68.2)
- added C50: 1uF, Capacitor_SMD:C_0603_1608Metric_Pad1.05x0.95mm_HandSolder, B.Cu at (136.8, 68.2)
- added C51: 1uF, Capacitor_SMD:C_0603_1608Metric_Pad1.05x0.95mm_HandSolder, B.Cu at (161.2, 68.2)
- added C52: 0.1uF, Capacitor_SMD:C_0603_1608Metric_Pad1.05x0.95mm_HandSolder, B.Cu at (218.5, 68.2)
- added C53: 0.1uF, Capacitor_SMD:C_0603_1608Metric_Pad1.05x0.95mm_HandSolder, B.Cu at (194.2, 68.2)
- added C54: 1uF, Capacitor_SMD:C_0603_1608Metric_Pad1.05x0.95mm_HandSolder, B.Cu at (208.5, 68.2)
- added C55: 1uF, Capacitor_SMD:C_0603_1608Metric_Pad1.05x0.95mm_HandSolder, B.Cu at (185.0, 68.2)
- added C7: 10uF, Capacitor_SMD:C_1210_3225Metric_Pad1.42x2.65mm_HandSolder, B.Cu at (77.0, 104.0)
- added D1: D_Schottky, BoringFootprints:DO-221AC, F.Cu at (72.0, 114.2)
- added D10: 1.5KExxCA, Diode_THT:D_DO-201AE_P15.24mm_Horizontal, F.Cu at (84.8, 45.5)
- added D11: 1.5KExxCA, Diode_THT:D_DO-201AE_P15.24mm_Horizontal, F.Cu at (96.8, 60.7)
- added D12: 1.5KExxCA, Diode_THT:D_DO-201AE_P15.24mm_Horizontal, F.Cu at (114.8, 45.5)
- added D13: 1.5KExxCA, Diode_THT:D_DO-201AE_P15.24mm_Horizontal, F.Cu at (120.8, 60.8)
- added D14: 1.5KExxCA, Diode_THT:D_DO-201AE_P15.24mm_Horizontal, F.Cu at (144.8, 60.8)
- added D15: 1.5KExxCA, Diode_THT:D_DO-201AE_P15.24mm_Horizontal, F.Cu at (132.8, 45.5)
- added D16: 1.5KExxCA, Diode_THT:D_DO-201AE_P15.24mm_Horizontal, F.Cu at (174.8, 60.8)
- added D17: 1.5KExxCA, Diode_THT:D_DO-201AE_P15.24mm_Horizontal, F.Cu at (156.8, 45.5)
- added D18: 1.5KExxCA, Diode_THT:D_DO-201AE_P15.24mm_Horizontal, F.Cu at (138.8, 45.5)
- added D19: 1.5KExxCA, Diode_THT:D_DO-201AE_P15.24mm_Horizontal, F.Cu at (150.8, 60.8)
- added D20: 1.5KExxCA, Diode_THT:D_DO-201AE_P15.24mm_Horizontal, F.Cu at (162.8, 45.5)
- added D21: 1.5KExxCA, Diode_THT:D_DO-201AE_P15.24mm_Horizontal, F.Cu at (168.8, 60.8)
- added D22: 1.5KExxCA, Diode_THT:D_DO-201AE_P15.24mm_Horizontal, F.Cu at (192.8, 60.8)
- added D23: 1.5KExxCA, Diode_THT:D_DO-201AE_P15.24mm_Horizontal, F.Cu at (216.8, 60.8)
- added D24: 1.5KExxCA, Diode_THT:D_DO-201AE_P15.24mm_Horizontal, F.Cu at (186.8, 45.5)
- added D25: 1.5KExxCA, Diode_THT:D_DO-201AE_P15.24mm_Horizontal, F.Cu at (204.8, 45.5)
- added D26: 1.5KExxCA, Diode_THT:D_DO-201AE_P15.24mm_Horizontal, F.Cu at (180.8, 45.5)
- added D27: 1.5KExxCA, Diode_THT:D_DO-201AE_P15.24mm_Horizontal, F.Cu at (210.8, 45.5)
- added D28: 1.5KExxCA, Diode_THT:D_DO-201AE_P15.24mm_Horizontal, F.Cu at (198.8, 60.8)
- added D29: 1.5KExxCA, Diode_THT:D_DO-201AE_P15.24mm_Horizontal, F.Cu at (222.8, 60.8)
- added D4: GREEN, LED_SMD:LED_0805_2012Metric_Pad1.15x1.40mm_HandSolder, B.Cu at (144.0, 118.8)
- added D5: BLUE, LED_SMD:LED_0805_2012Metric_Pad1.15x1.40mm_HandSolder, B.Cu at (141.2, 94.5)
- added D6: 1.5KExxCA, Diode_THT:D_DO-201AE_P15.24mm_Horizontal, F.Cu at (102.8, 60.8)
- added D7: 1.5KExxCA, Diode_THT:D_DO-201AE_P15.24mm_Horizontal, F.Cu at (90.8, 45.5)
- added D8: 1.5KExxCA, Diode_THT:D_DO-201AE_P15.24mm_Horizontal, F.Cu at (126.8, 60.8)
- added D9: 1.5KExxCA, Diode_THT:D_DO-201AE_P15.24mm_Horizontal, F.Cu at (108.8, 45.5)
- added F1: Fuse, BoringFootprints:BelFuse_0679H, F.Cu at (65.0, 114.2)
- added G***: LOGO, BoringFootprints:Paradigm_NameBelow_25.4mm, F.Cu at (208.8, 99.2)
- added J1: Conn_01x12, Connector_Molex:Molex_Micro-Fit_3.0_43045-1200_2x06_P3.00mm_Horizontal, F.Cu at (59.5, 110.8)
- added J10: PRESS_9, Connector_Molex:Molex_Nano-Fit_105313-xx03_1x03_P2.50mm_Horizontal, F.Cu at (162.2, 139.2)
- added J11: PRESS_10, Connector_Molex:Molex_Nano-Fit_105313-xx03_1x03_P2.50mm_Horizontal, F.Cu at (152.8, 139.2)
- added J12: FLAMM_1, Connector_Molex:Molex_Micro-Fit_3.0_43045-0400_2x02_P3.00mm_Horizontal, F.Cu at (141.2, 140.8)
- added J13: FLAMM_2, Connector_Molex:Molex_Micro-Fit_3.0_43045-0400_2x02_P3.00mm_Horizontal, F.Cu at (130.0, 140.8)
- added J14: TEMPRESS_1, Connector_Molex:Molex_Micro-Fit_3.0_43045-0400_2x02_P3.00mm_Horizontal, F.Cu at (118.8, 140.8)
- added J15: TEMPRESS_2, Connector_Molex:Molex_Micro-Fit_3.0_43045-0400_2x02_P3.00mm_Horizontal, F.Cu at (107.5, 140.8)
- added J16: TEMPRESS_3, Connector_Molex:Molex_Micro-Fit_3.0_43045-0400_2x02_P3.00mm_Horizontal, F.Cu at (96.2, 140.8)
- added J17: TEMPRESS_4, Connector_Molex:Molex_Micro-Fit_3.0_43045-0400_2x02_P3.00mm_Horizontal, F.Cu at (85.0, 140.8)
- added J18: TACH_1, Connector_Molex:Molex_Micro-Fit_3.0_43650-0300_1x03_P3.00mm_Horizontal, F.Cu at (74.0, 140.8)
- added J19: TACH_2, Connector_Molex:Molex_Micro-Fit_3.0_43650-0300_1x03_P3.00mm_Horizontal, F.Cu at (60.2, 140.8)
- added J2: PRESS_1, Connector_Molex:Molex_Nano-Fit_105313-xx03_1x03_P2.50mm_Horizontal, F.Cu at (238.2, 139.2)
- added J20: Conn_01x02, Connector_Molex:Molex_Micro-Fit_3.0_43045-0200_2x01_P3.00mm_Horizontal, F.Cu at (87.8, 39.5)
- added J21: Conn_01x02, Connector_Molex:Molex_Micro-Fit_3.0_43045-0200_2x01_P3.00mm_Horizontal, F.Cu at (99.8, 39.5)
- added J22: Conn_01x02, Connector_Molex:Molex_Micro-Fit_3.0_43045-0200_2x01_P3.00mm_Horizontal, F.Cu at (111.8, 39.5)
- added J23: Conn_01x02, Connector_Molex:Molex_Micro-Fit_3.0_43045-0200_2x01_P3.00mm_Horizontal, F.Cu at (123.8, 39.5)
- added J24: Conn_01x02, Connector_Molex:Molex_Micro-Fit_3.0_43045-0200_2x01_P3.00mm_Horizontal, F.Cu at (135.8, 39.5)
- added J25: Conn_01x02, Connector_Molex:Molex_Micro-Fit_3.0_43045-0200_2x01_P3.00mm_Horizontal, F.Cu at (147.8, 39.5)
- added J26: Conn_01x02, Connector_Molex:Molex_Micro-Fit_3.0_43045-0200_2x01_P3.00mm_Horizontal, F.Cu at (159.8, 39.5)
- added J27: Conn_01x02, Connector_Molex:Molex_Micro-Fit_3.0_43045-0200_2x01_P3.00mm_Horizontal, F.Cu at (171.8, 39.5)
- added J28: Conn_01x02, Connector_Molex:Molex_Micro-Fit_3.0_43045-0200_2x01_P3.00mm_Horizontal, F.Cu at (183.8, 39.5)
- added J29: Conn_01x02, Connector_Molex:Molex_Micro-Fit_3.0_43045-0200_2x01_P3.00mm_Horizontal, F.Cu at (195.8, 39.5)
- added J3: PRESS_2, Connector_Molex:Molex_Nano-Fit_105313-xx03_1x03_P2.50mm_Horizontal, F.Cu at (228.8, 139.2)
- added J30: Conn_01x02, Connector_Molex:Molex_Micro-Fit_3.0_43045-0200_2x01_P3.00mm_Horizontal, F.Cu at (207.8, 39.5)
- added J31: Conn_01x02, Connector_Molex:Molex_Micro-Fit_3.0_43045-0200_2x01_P3.00mm_Horizontal, F.Cu at (219.8, 39.5)
- added J4: PRESS_3, Connector_Molex:Molex_Nano-Fit_105313-xx03_1x03_P2.50mm_Horizontal, F.Cu at (219.2, 139.2)
- added J5: PRESS_4, Connector_Molex:Molex_Nano-Fit_105313-xx03_1x03_P2.50mm_Horizontal, F.Cu at (209.8, 139.2)
- added J6: PRESS_5, Connector_Molex:Molex_Nano-Fit_105313-xx03_1x03_P2.50mm_Horizontal, F.Cu at (200.2, 139.2)
- added J7: PRESS_6, Connector_Molex:Molex_Nano-Fit_105313-xx03_1x03_P2.50mm_Horizontal, F.Cu at (190.8, 139.2)
- added J8: PRESS_7, Connector_Molex:Molex_Nano-Fit_105313-xx03_1x03_P2.50mm_Horizontal, F.Cu at (181.2, 139.2)
- added J9: PRESS_8, Connector_Molex:Molex_Nano-Fit_105313-xx03_1x03_P2.50mm_Horizontal, F.Cu at (171.8, 139.2)
- added JP1: CAN_TERM, Jumper:SolderJumper-2_P1.3mm_Open_RoundedPad1.0x1.5mm, F.Cu at (88.2, 102.0)
- added R1: 1.1K, Resistor_SMD:R_0603_1608Metric_Pad1.05x0.95mm_HandSolder, B.Cu at (72.5, 95.2)
- added R10: DNP, Resistor_SMD:R_0603_1608Metric_Pad1.05x0.95mm_HandSolder, B.Cu at (151.5, 119.5)
- added R11: DNP, Resistor_SMD:R_0603_1608Metric_Pad1.05x0.95mm_HandSolder, B.Cu at (151.5, 121.2)
- added R12: DNP, Resistor_SMD:R_0603_1608Metric_Pad1.05x0.95mm_HandSolder, B.Cu at (155.0, 116.0)
- added R14: DNP, Resistor_SMD:R_0603_1608Metric_Pad1.05x0.95mm_HandSolder, B.Cu at (155.0, 119.5)
- added R15: DNP, Resistor_SMD:R_0603_1608Metric_Pad1.05x0.95mm_HandSolder, B.Cu at (155.0, 121.2)
- added R16: 47K, Resistor_SMD:R_0603_1608Metric_Pad1.05x0.95mm_HandSolder, B.Cu at (153.5, 104.2)
- added R17: 1K, Resistor_SMD:R_0603_1608Metric_Pad1.05x0.95mm_HandSolder, F.Cu at (144.0, 118.8)
- added R18: 1M, Resistor_SMD:R_0603_1608Metric_Pad1.05x0.95mm_HandSolder, B.Cu at (151.5, 98.0)
- added R19: 280K, Resistor_SMD:R_0603_1608Metric_Pad1.05x0.95mm_HandSolder, B.Cu at (154.8, 100.2)
- added R2: 240, Resistor_SMD:R_0603_1608Metric_Pad1.05x0.95mm_HandSolder, B.Cu at (72.5, 93.5)
- added R20: 604K, Resistor_SMD:R_0603_1608Metric_Pad1.05x0.95mm_HandSolder, B.Cu at (158.2, 97.5)
- added R21: 47K, Resistor_SMD:R_0603_1608Metric_Pad1.05x0.95mm_HandSolder, B.Cu at (150.8, 90.0)
- added R22: 47K, Resistor_SMD:R_0603_1608Metric_Pad1.05x0.95mm_HandSolder, B.Cu at (145.8, 93.5)
- added R23: 1K, Resistor_SMD:R_0603_1608Metric_Pad1.05x0.95mm_HandSolder, F.Cu at (141.2, 94.5)
- added R24: 1K, Resistor_SMD:R_0603_1608Metric_Pad1.05x0.95mm_HandSolder, F.Cu at (235.8, 135.8)
- added R25: 1K, Resistor_SMD:R_0603_1608Metric_Pad1.05x0.95mm_HandSolder, F.Cu at (226.2, 135.8)
- added R26: 1K, Resistor_SMD:R_0603_1608Metric_Pad1.05x0.95mm_HandSolder, F.Cu at (216.8, 135.8)
- added R27: 1K, Resistor_SMD:R_0603_1608Metric_Pad1.05x0.95mm_HandSolder, F.Cu at (207.2, 135.8)
- added R28: 1K, Resistor_SMD:R_0603_1608Metric_Pad1.05x0.95mm_HandSolder, F.Cu at (197.8, 135.8)
- added R29: 1K, Resistor_SMD:R_0603_1608Metric_Pad1.05x0.95mm_HandSolder, F.Cu at (188.2, 135.8)
- added R3: 0, Resistor_SMD:R_0603_1608Metric_Pad1.05x0.95mm_HandSolder, F.Cu at (162.8, 111.2)
- added R30: 1K, Resistor_SMD:R_0603_1608Metric_Pad1.05x0.95mm_HandSolder, F.Cu at (178.8, 135.8)
- added R31: 1K, Resistor_SMD:R_0603_1608Metric_Pad1.05x0.95mm_HandSolder, F.Cu at (169.2, 135.8)
- added R32: 10K, Resistor_SMD:R_0603_1608Metric_Pad1.05x0.95mm_HandSolder, F.Cu at (129.5, 127.8)
- added R33: 22K, Resistor_SMD:R_0603_1608Metric_Pad1.05x0.95mm_HandSolder, F.Cu at (129.5, 129.2)
- added R34: 1K, Resistor_SMD:R_0603_1608Metric_Pad1.05x0.95mm_HandSolder, F.Cu at (159.8, 135.8)
- added R35: 1K, Resistor_SMD:R_0603_1608Metric_Pad1.05x0.95mm_HandSolder, F.Cu at (150.2, 135.8)
- added R36: 10K, Resistor_SMD:R_0603_1608Metric_Pad1.05x0.95mm_HandSolder, F.Cu at (141.2, 134.5)
- added R37: 10K, Resistor_SMD:R_0603_1608Metric_Pad1.05x0.95mm_HandSolder, F.Cu at (130.0, 134.5)
- added R38: 10K, Resistor_SMD:R_0603_1608Metric_Pad1.05x0.95mm_HandSolder, F.Cu at (118.8, 134.5)
- added R39: 10K, Resistor_SMD:R_0603_1608Metric_Pad1.05x0.95mm_HandSolder, F.Cu at (107.5, 134.5)
- added R4: 0, Resistor_SMD:R_0603_1608Metric_Pad1.05x0.95mm_HandSolder, F.Cu at (157.0, 114.0)
- added R40: 10K, Resistor_SMD:R_0603_1608Metric_Pad1.05x0.95mm_HandSolder, F.Cu at (96.2, 134.5)
- added R41: 10K, Resistor_SMD:R_0603_1608Metric_Pad1.05x0.95mm_HandSolder, F.Cu at (85.0, 134.5)
- added R42: 1K, Resistor_SMD:R_0603_1608Metric_Pad1.05x0.95mm_HandSolder, F.Cu at (115.8, 134.5)
- added R43: 1K, Resistor_SMD:R_0603_1608Metric_Pad1.05x0.95mm_HandSolder, F.Cu at (104.5, 134.5)
- added R44: 1K, Resistor_SMD:R_0603_1608Metric_Pad1.05x0.95mm_HandSolder, F.Cu at (93.2, 134.5)
- added R45: 1K, Resistor_SMD:R_0603_1608Metric_Pad1.05x0.95mm_HandSolder, F.Cu at (82.0, 134.5)
- added R46: 10K, Resistor_SMD:R_0603_1608Metric_Pad1.05x0.95mm_HandSolder, F.Cu at (69.5, 137.0)
- added R47: 10K, Resistor_SMD:R_0603_1608Metric_Pad1.05x0.95mm_HandSolder, F.Cu at (55.8, 137.0)
- added R5: 0, Resistor_SMD:R_0603_1608Metric_Pad1.05x0.95mm_HandSolder, F.Cu at (154.0, 109.5)
- added R6: 0, Resistor_SMD:R_0603_1608Metric_Pad1.05x0.95mm_HandSolder, F.Cu at (157.0, 106.8)
- added R7: 120, Resistor_SMD:R_1210_3225Metric_Pad1.42x2.65mm_HandSolder, F.Cu at (88.2, 106.0)
- added R8: DNP, Resistor_SMD:R_0603_1608Metric_Pad1.05x0.95mm_HandSolder, B.Cu at (151.5, 116.0)
- added R9: DNP, Resistor_SMD:R_0603_1608Metric_Pad1.05x0.95mm_HandSolder, B.Cu at (151.5, 117.8)
- added REF**: Paradigm_Title_Block, BoringFootprints:Paradigm_Title_Block, F.Cu at (240.5, 65.5)
- added REF**: MountingHole_3.2mm_M3, MountingHole:MountingHole_3.2mm_M3, F.Cu at (54.0, 69.2)
- added REF**: MountingHole_3.2mm_M3, MountingHole:MountingHole_3.2mm_M3, F.Cu at (54.0, 129.5)
- added REF**: MountingHole_3.2mm_M3, MountingHole:MountingHole_3.2mm_M3, F.Cu at (246.0, 34.0)
- added REF**: MountingHole_3.2mm_M3, MountingHole:MountingHole_3.2mm_M3, F.Cu at (246.0, 146.0)
- added REF**: MountingHole_3.2mm_M3, MountingHole:MountingHole_3.2mm_M3, F.Cu at (54.0, 34.0)
- added U10: LM2902, Package_SO:SOIC-14_3.9x8.7mm_P1.27mm, F.Cu at (135.2, 127.8)
- added U11: ADC128S022, Package_SO:TSSOP-16_4.4x5mm_P0.65mm, F.Cu at (202.7, 123.7)
- added U12: ADC128S022, Package_SO:TSSOP-16_4.4x5mm_P0.65mm, F.Cu at (92.2, 122.5)
- added U13: L293D, Package_DIP:DIP-16_W7.62mm, F.Cu at (102.5, 64.0)
- added U14: L293D, Package_DIP:DIP-16_W7.62mm, F.Cu at (126.8, 64.0)
- added U15: L293D, Package_DIP:DIP-16_W7.62mm, F.Cu at (150.5, 64.0)
- added U16: L293D, Package_DIP:DIP-16_W7.62mm, F.Cu at (174.8, 64.0)
- added U17: L293D, Package_DIP:DIP-16_W7.62mm, F.Cu at (198.5, 64.0)
- added U18: L293D, Package_DIP:DIP-16_W7.62mm, F.Cu at (222.2, 64.0)
- added U8: 74LVC1G17, Package_TO_SOT_SMD:SOT-23-5_HandSoldering, B.Cu at (141.2, 91.2)
- added U9: LTC6993xS6-1, Package_TO_SOT_SMD:TSOT-23-6, B.Cu at (154.8, 97.5)
- C1: value 0.1uF -> 1uF; moved to B.Cu
- C2, C3, C5, C6: value 0.1uF -> 10uF; footprint Capacitor_SMD:C_0603_1608Metric_Pad1.05x0.95mm_HandSolder -> Capacitor_SMD:C_1210_3225Metric_Pad1.42x2.65mm_HandSolder
- C4, C8, Q1, Q2, U4: moved to B.Cu
- D2: value GREEN -> 1N4002; footprint LED_SMD:LED_0805_2012Metric_Pad1.15x1.40mm_HandSolder -> Package_TO_SOT_SMD:SOT-23_Handsoldering
- D3: value BLUE -> 1N4002; footprint LED_SMD:LED_0805_2012Metric_Pad1.15x1.40mm_HandSolder -> Package_TO_SOT_SMD:SOT-23_Handsoldering; moved to B.Cu
- R13: value 120 -> DNP; moved to B.Cu
- U1: value 74HC21 -> R-78B12-2.0; footprint Package_SO:SOIC-14_3.9x8.7mm_P1.27mm -> Converter_DCDC:Converter_DCDC_RECOM_R-78B-2.0_THT
- U2: value 74HC266 -> LM317DCYRG3; footprint Package_SO:SOIC-14_3.9x8.7mm_P1.27mm -> Package_TO_SOT_SMD:SOT-223-3_TabPin2
- U3: value 74HC08 -> SN65HVD232; footprint Package_SO:SOIC-14_3.9x8.7mm_P1.27mm -> Package_SO:SOIC-8_3.9x4.9mm_P1.27mm
- U5: value 74LVC1G17 -> 74HC266; footprint Package_TO_SOT_SMD:SOT-23-5_HandSoldering -> Package_SO:SOIC-14_3.9x8.7mm_P1.27mm; moved to B.Cu
- U6: value LTC6993xS6-1 -> 74HC08; footprint Package_TO_SOT_SMD:TSOT-23-6 -> Package_SO:SOIC-14_3.9x8.7mm_P1.27mm; moved to B.Cu
- U7: value SN65HVD232 -> 74HC21; footprint Package_SO:SOIC-8_3.9x4.9mm_P1.27mm -> Package_SO:SOIC-14_3.9x8.7mm_P1.27mm; moved to B.Cu
- moved C9 193.3 mm to (69.8, 94.5), turned to 90 degrees
- moved R13 97.4 mm to (155.0, 117.8), turned to 180 degrees
- moved U7 96.0 mm to (133.8, 110.0), turned to 180 degrees
- moved Q1 92.2 mm to (150.8, 92.8), turned to 0 degrees
- moved C2 90.4 mm to (186.5, 100.2)
- moved Q2 89.8 mm to (145.8, 89.8)
- moved C3 80.9 mm to (186.5, 103.5)
- moved C5 80.7 mm to (186.5, 106.8)
- moved U6 77.8 mm to (141.5, 110.0), turned to 180 degrees
- moved C6 75.2 mm to (186.5, 110.0)
- moved U4 66.5 mm to (157.0, 110.0), turned to 180 degrees
- moved C8 64.0 mm to (76.0, 95.2), turned to 180 degrees
- moved U5 47.8 mm to (149.2, 110.0), turned to 180 degrees
- moved NCLO1 45.2 mm to (178.5, 82.0), turned to 180 degrees
- moved U1 44.0 mm to (71.5, 108.8), turned to 90 degrees
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Connections:
- C1 pad 1: +5V -> +24V
- C2 pad 1: +5V -> +12V
- C3 pad 1: +5V -> +12V
- C4 pad 1: +5V -> +12V
- C5 pad 1: +5V -> +12V
- C6 pad 1: +5V -> +12V
- C8 pad 1: +3V3 -> +12V
- C9 pad 1: /Acquisition/ANALOG_IN_1 -> Net-(C9-Pad1)
- D2 pad 1: Net-(D2-Pad1) -> +12V
- D2 pad 2: Net-(D2-Pad2) -> 7V
- D3 pad 1: Net-(D3-Pad1) -> 7V
- D3 pad 2: /HEARTBEAT_BUFF -> Net-(C9-Pad1)
- NCLO1 pad 1: Net-(NCLO1-Pad1) -> /ACT_IN_6
- NCLO1 pad 13: Net-(NCLO1-Pad13) -> /HEARTBEAT_BUFF
- NCLO1 pad 15: Net-(NCLO1-Pad15) -> /ACT_EN_8
- NCLO1 pad 2: Net-(NCLO1-Pad2) -> /ACT_IN_5
- NCLO1 pad 21: Net-(NCLO1-Pad21) -> /ACT_IN_21
- NCLO1 pad 23: Net-(NCLO1-Pad23) -> /ACT_IN_3
- NCLO1 pad 25: Net-(NCLO1-Pad25) -> /ACT_IN_2
- NCLO1 pad 27: Net-(NCLO1-Pad27) -> /ACT_IN_1
- NCLO1 pad 28: /HEARTBEAT_BUFF -> /TEMP_1
- NCLO1 pad 3: Net-(NCLO1-Pad3) -> /ACT_IN_4
- NCLO1 pad 30: Net-(NCLO1-Pad30) -> /TEMP_2
- NCLO1 pad 32: Net-(NCLO1-Pad32) -> /ACT_EN_2
- NCLO1 pad 35: Net-(NCLO1-Pad35) -> /ACT_IN_14
- NCLO1 pad 36: Net-(NCLO1-Pad36) -> /ACT_IN_15
- NCLO1 pad 37: Net-(NCLO1-Pad37) -> /ACT_IN_13
- NCLO1 pad 38: Net-(NCLO1-Pad38) -> /ACT_IN_16
- NCLO1 pad 39: Net-(NCLO1-Pad39) -> /ACT_IN_7
- NCLO1 pad 40: Net-(NCLO1-Pad40) -> /ACT_IN_8
- NCLO1 pad 41: Net-(NCLO1-Pad41) -> /ACT_IN_22
- NCLO1 pad 42: Net-(NCLO1-Pad42) -> /ACT_IN_10
- NCLO1 pad 43: Net-(NCLO1-Pad43) -> /ACT_IN_23
- NCLO1 pad 44: Net-(NCLO1-Pad44) -> /ACT_IN_11
- NCLO1 pad 49: Net-(NCLO1-Pad49) -> /ACT_EN_1
- NCLO1 pad 51: Net-(NCLO1-Pad51) -> /TEMP_3
- NCLO1 pad 53: Net-(NCLO1-Pad53) -> /TEMP_4
- NCLO1 pad 54: Net-(NCLO1-Pad54) -> /ADC2_nCS
- NCLO1 pad 55: Net-(NCLO1-Pad55) -> /ACT_IN_20
- NCLO1 pad 56: Net-(NCLO1-Pad56) -> /ADC1_nCS
- NCLO1 pad 57: Net-(NCLO1-Pad57) -> /ACT_IN_9
- NCLO1 pad 59: Net-(NCLO1-Pad59) -> /ACT_EN_6
- NCLO1 pad 60: Net-(NCLO1-Pad60) -> /HEARTBEAT_RESTART
- NCLO1 pad 61: Net-(NCLO1-Pad61) -> /ACT_EN_7
- NCLO1 pad 62: Net-(NCLO1-Pad62) -> /MCU_QB_INPUT
- NCLO1 pad 63: Net-(NCLO1-Pad63) -> /ACT_IN_24
- NCLO1 pad 64: Net-(NCLO1-Pad64) -> /SPI_MOSI
- NCLO1 pad 65: Net-(NCLO1-Pad65) -> /ACT_IN_18
- NCLO1 pad 66: Net-(NCLO1-Pad66) -> /SPI_MISO
- NCLO1 pad 67: Net-(NCLO1-Pad67) -> /ACT_IN_19
- NCLO1 pad 68: Net-(NCLO1-Pad68) -> /SPI_SCLK
- NCLO1 pad 69: Net-(NCLO1-Pad69) -> /ACT_IN_17
- NCLO1 pad 71: Net-(NCLO1-Pad71) -> /ACT_EN_5
- NCLO1 pad 72: Net-(NCLO1-Pad72) -> /ACT_IN_12
- NCLO1 pad 73: Net-(NCLO1-Pad73) -> /ACT_EN_4
- NCLO1 pad 75: Net-(NCLO1-Pad75) -> /ACT_EN_3
- R13 pad 1: Net-(JP1-Pad1) -> +5V
- R13 pad 2: /CANH -> Net-(R13-Pad2)
- U1 pad 1: /AvionicsHeartbeatTemplate/HEARTBEAT_INPUT_1 -> +24V
- U1 pad 2: /AvionicsHeartbeatTemplate/HEARTBEAT_INPUT_2 -> GND
- U1 pad 3: (no net) -> +12V
- U2 pad 1: /HEARTBEAT_ADDRESS_4 -> Net-(C9-Pad1)
- U2 pad 2: Net-(R1-Pad2) -> 7V
- U2 pad 3: Net-(U2-Pad3) -> +12V
- U3 pad 1: Net-(U1-Pad6) -> /CAN_TX
- U3 pad 2: Net-(U1-Pad8) -> GND
- U3 pad 3: Net-(D2-Pad2) -> +3V3
- U3 pad 4: Net-(D2-Pad2) -> /CAN_RX
- U3 pad 6: Net-(U3-Pad6) -> /CANL
- U3 pad 7: GND -> /CANH
- U3 pad 8: (no net) -> Net-(U3-Pad8)
- U4 pad 1: Net-(U2-Pad3) -> /MCU_QB_INPUT
- U4 pad 10: (no net) -> /AvionicsHeartbeatTemplate/HEARTBEAT_INPUT_6
- U4 pad 12: (no net) -> /AvionicsHeartbeatTemplate/HEARTBEAT_INPUT_7
- U4 pad 13: (no net) -> /HEARTBEAT_RESTART
- U4 pad 2: Net-(U2-Pad4) -> /FLAMM_SAFE_1
- U4 pad 4: Net-(U2-Pad10) -> /FLAMM_SAFE_2
- U4 pad 5: Net-(U2-Pad11) -> /AvionicsHeartbeatTemplate/HEARTBEAT_INPUT_4
- U4 pad 6: Net-(U3-Pad5) -> Net-(U4-Pad6)
- U4 pad 8: (no net) -> Net-(U4-Pad8)
- U4 pad 9: (no net) -> /AvionicsHeartbeatTemplate/HEARTBEAT_INPUT_5
- U5 pad 1: (no net) -> /HEARTBEAT_ADDRESS_4
- U5 pad 2: /HEARTBEAT -> Net-(R12-Pad2)
- U5 pad 3: GND -> Net-(U5-Pad3)
- U5 pad 4: /HEARTBEAT_BUFF -> Net-(U5-Pad4)
- U5 pad 5: +5V -> /HEARTBEAT_ADDRESS_3
- U6 pad 1: Net-(U3-Pad6) -> Net-(U4-Pad6)
- U6 pad 2: GND -> Net-(U4-Pad8)
- U6 pad 3: Net-(R11-Pad1) -> Net-(D4-Pad2)
- U6 pad 4: Net-(R10-Pad1) -> Net-(D4-Pad2)
- U6 pad 5: +5V -> Net-(U6-Pad5)
- U6 pad 6: Net-(Q1-Pad1) -> Net-(U6-Pad6)
- U7 pad 1: /CAN_TX -> Net-(U5-Pad3)
- U7 pad 2: GND -> Net-(U5-Pad4)
- U7 pad 3: +3V3 -> (no net)
- U7 pad 4: /CAN_RX -> Net-(U5-Pad10)
- U7 pad 5: Net-(U7-Pad5) -> Net-(U5-Pad11)
- U7 pad 6: /CANL -> Net-(U6-Pad5)
- U7 pad 7: /CANH -> GND
- U7 pad 8: Net-(U7-Pad8) -> (no net)
Routing:
- net GND: track 0.00 -> 153.1 mm, vias 0 -> 13
- net +24V: track 0.00 -> 77.0 mm, vias 0 -> 6
- net Net-(D23-Pad2): track 0.00 -> 62.0 mm
- net Net-(D11-Pad2): track 0.00 -> 58.9 mm
- net /Acquisition/FLAMM_2: track 0.00 -> 58.0 mm
- net /Acquisition/FLAMM_1: track 0.00 -> 56.0 mm
- net Net-(D22-Pad2): track 0.00 -> 52.3 mm
- net Net-(D14-Pad2): track 0.00 -> 52.0 mm
- net Net-(D21-Pad2): track 0.00 -> 47.4 mm
- net Net-(D29-Pad2): track 0.00 -> 46.6 mm
- net Net-(D19-Pad2): track 0.00 -> 45.0 mm
- net Net-(D28-Pad2): track 0.00 -> 45.0 mm
- net Net-(D13-Pad2): track 0.00 -> 43.8 mm
- net /Acquisition/PRESS_1: track 0.00 -> 43.4 mm
- net /Acquisition/PRESS_8: track 0.00 -> 42.4 mm
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- added copper zone on B.Cu, net (none)
- added copper zone on B.Cu, net +24V
- added copper zone on B.Cu, net GND
Other:
- board outline added: 200 x 120 mm
- board text added: "A"
- board text added: "PLV002_THOR"
- board text added: "Thor Sensor/Actuator Board"
