File: PCB_PLV002_Thor/AvionicsHeartbeat.sch (KiCad schematic (older format))
At the start: 33 parts, among them Q1 DMG2302UK-7, Q2 DMP2123L-7, U1 74HC21, U2 74HC266, U3 74HC08, U4 74HC21, U5 74LVC1G17, U6 LTC6993xS6-1

Commit message: Done
Parts:
- renumbered C1 to C12, C2 to C13, C3 to C14, C4 to C15, C5 to C16, C6 to C17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
