File: PCB_PLV005_Beyla/PCB_PLV005_Beyla.kicad_pcb (KiCad board)
At the start: 2 copper layers, 50 x 50 mm, 44 parts, among them J1 PWR/QB, J2 Switch_In, Q1 DMG2302UK-7, Q2 DMP2123L-7, U2 74HC266, U3 74HC08, U4 74HC21, U5 74LVC1G17, U6 LTC6993xS6-1

Commit message: Beyla Voltage Regulator Fix
Connections:
- VR1 pad 1: +5V -> Net-(C8-Pad1)
- VR1 pad 3: Net-(C8-Pad1) -> +5V
Routing:
- net GND: track 58.7 -> 53.5 mm, vias 15 -> 16
- net Net-(C8-Pad1): track 91.5 -> 96.7 mm, vias 0 -> 1
- net +5V: track 165.8 -> 170.7 mm
- net Net-(D1-Pad1): track 17.0 -> 12.5 mm
