File: PCB_PLV008_Loki/Acquisition.sch (KiCad schematic (older format))
At the start: 18 parts

Commit message: Add files via upload
Parts:
- removed 3.4V, 3.4V? (x2): D_Zener, symbol Device:D_Zener
- removed C? (x2): 0.1uF, symbol Device:C
- removed J? (x2): Conn_01x03, symbol Connector_Generic:Conn_01x03
- removed R? (x3): 10K, symbol Device:R_US
- removed R? (x2): 1K, symbol Device:R_US
- removed U? (x3): LM2902, symbol Amplifier_Operational:LM2902
- added C19, C20, C21, C22, C23, C24, C25, C26, C27, C28, C29, C30, C31, C32, C33, C34, C35, C36, C37, C38, C39, C40, C41, C42, C43, C50, C51, C52, C53, C54, C55: 0.1uF, symbol Device:C
- added C44, C45, C46, C47, C48, C49: 1uF, symbol Device:C
- added J10, J16, J17, J18, J19, J21, J22, J8, J9: Conn_01x04, symbol Connector_Generic:Conn_01x04
- added J11, J12, J13, J14, J2, J3, J4, J5, J6, J7: Conn_01x03, symbol Connector_Generic:Conn_01x03
- added J15: Conn_01x08, symbol Connector_Generic:Conn_01x08
- added J20: Conn_01x06, symbol Connector_Generic:Conn_01x06
- added R18, R19, R20, R21, R22, R23, R24, R32, R33, R34, R35: 100, symbol Device:R_US
- added R26, R27, R28, R29, R30, R31, R39, R40, R41, R42, R43, R44, R45, R53, R54, R55, R56, R57, R58, R59, R65, R66, R67, R68, R69: 1K, symbol Device:R_US
- added R36, R37, R38, R46, R47, R48, R49, R50, R51, R52, R60, R61, R62, R63, R64: 516, symbol Device:R_US
- added U5, U6, U7: ADC128S022CIMT, SOP65P640X120-16N, symbol ADC128S022CIMT:ADC128S022CIMT
- gave numbers to parts that had none: 3
Connections:
- net +3V3: now also C44.1, C46.1, C48.1, C50.1, C52.1, C54.1, J11.1 (Pin_1), J12.1 (Pin_1), J13.1 (Pin_1), J14.1 (Pin_1), J2.1 (Pin_1), J3.1 (Pin_1), J4.1 (Pin_1), J5.1 (Pin_1), J6.1 (Pin_1), J7.1 (Pin_1), U5.13 (VD), U6.13 (VD), U7.13 (VD)
- net GND: now also C19.2, C20.2, C21.2, C22.2, C23.2, C24.2, C25.2, C26.2, C27.2, C28.2, C29.2, C30.2, C31.2, C32.2, C33.2, C34.2, C35.2, C36.2, C37.2, C38.2, C39.2, C40.2, C41.2, C42.2, C43.2, C44.2, C45.2, C46.2, C47.2, C48.2, C49.2, C50.2, C51.2, C52.2, C53.2, C54.2, C55.2, J10.3 (Pin_3), J10.4 (Pin_4), J11.3 (Pin_3), J12.3 (Pin_3), J13.3 (Pin_3), J14.3 (Pin_3), J15.2 (Pin_2), J15.4 (Pin_4), J15.6 (Pin_6), J15.8 (Pin_8), J16.3 (Pin_3), J16.4 (Pin_4), J17.3 (Pin_3), J17.4 (Pin_4), J18.3 (Pin_3), J18.4 (Pin_4), J19.3 (Pin_3), J19.4 (Pin_4), J2.3 (Pin_3), J20.5 (Pin_5), J20.6 (Pin_6), J21.3 (Pin_3), J21.4 (Pin_4), J22.3 (Pin_3), J22.4 (Pin_4), J3.3 (Pin_3), J4.3 (Pin_3), J5.3 (Pin_3), J6.3 (Pin_3), J7.3 (Pin_3), J8.3 (Pin_3), J8.4 (Pin_4), J9.3 (Pin_3), J9.4 (Pin_4), R18.2, R19.2, R20.2, R21.2, R22.2, R23.2, R24.2, R32.2, R33.2, R34.2, R35.2, R36.2, R37.2, R38.2, R46.2, R47.2, R48.2, R49.2, R50.2, R51.2, R52.2, R60.2, R61.2, R62.2, R63.2, R64.2, U5.12 (DGND), U5.3 (AGND), U6.12 (DGND), U6.3 (AGND), U7.12 (DGND), U7.3 (AGND)
- net at R25.1: now also J1.2 (Pin_2), R18.1
- net STemp1: now reaches C18.1, R25.2
- net STemp1: now also U5.4 (IN0)
- new net: J10.2 (Pin_2), R38.1, R45.1
- new net: J2.2 (Pin_2), R19.1, R26.1
- new net: J3.2 (Pin_2), R20.1, R27.1
- new net: J4.2 (Pin_2), R21.1, R28.1
- new net: J5.2 (Pin_2), R22.1, R29.1
- new net: J6.2 (Pin_2), R23.1, R30.1
- new net: J7.2 (Pin_2), R24.1, R31.1
- new net: J11.2 (Pin_2), R32.1, R39.1
- new net: J12.2 (Pin_2), R33.1, R40.1
- new net: J13.2 (Pin_2), R34.1, R41.1
- new net: J14.2 (Pin_2), R35.1, R42.1
- new net: J8.2 (Pin_2), R36.1, R43.1
- new net: J9.2 (Pin_2), R37.1, R44.1
- new net: J15.3 (Pin_3), R46.1, R53.1
- new net: J15.5 (Pin_5), R47.1, R54.1
- new net: J15.7 (Pin_7), R48.1, R55.1
- new net: J16.2 (Pin_2), R49.1, R56.1
- new net: J17.2 (Pin_2), R50.1, R57.1
- new net: J18.2 (Pin_2), R51.1, R58.1
- new net: J19.2 (Pin_2), R52.1, R59.1
- new net: J20.2 (Pin_2), R60.1, R65.1
- new net: J20.3 (Pin_3), R61.1, R66.1
- new net: J20.4 (Pin_4), R62.1, R67.1
- new net: J21.2 (Pin_2), R63.1, R68.1
- new net: J22.2 (Pin_2), R64.1, R69.1
- new net +12V: J10.1 (Pin_1), J15.1 (Pin_1), J16.1 (Pin_1), J17.1 (Pin_1), J18.1 (Pin_1), J19.1 (Pin_1), J20.1 (Pin_1), J21.1 (Pin_1), J22.1 (Pin_1), J8.1 (Pin_1), J9.1 (Pin_1)
- new net +5V: C45.1, C47.1, C49.1, C51.1, C53.1, C55.1, U5.2 (VA), U6.2 (VA), U7.2 (VA)
- new net 3ACCU1: C32.1, R53.2, U7.10 (IN6)
- new net 3ACCU2: C33.1, R54.2, U7.11 (IN7)
- new net 3ACCU3: C34.1, R55.2, U6.4 (IN0)
- new net 3ACVO1: C39.1, R65.2, U6.9 (IN5)
- new net 3ACVO2: C40.1, R66.2, U6.10 (IN6)
- new net 3ACVO3: C41.1, R67.2, U6.11 (IN7)
- new net ACCU1: C31.1, R45.2, U7.7 (IN3)
- new net ACCU2: C29.1, R43.2, U7.8 (IN4)
- new net ACVO1: C42.1, R68.2
- new net ACVO2: C43.1, R69.2
- new net DCCU1: C30.1, R44.2, U7.9 (IN5)
- new net DCVO1: C38.1, R59.2, U6.8 (IN4)
- new net DOUT: U5.15 (DOUT), U6.15 (DOUT), U7.15 (DOUT)
- new net DataIn: U5.14 (DIN), U6.14 (DIN), U7.14 (DIN)
- new net GFO1: C35.1, R56.2, U6.5 (IN1)
- new net GFO2: C36.1, R57.2, U6.6 (IN2)
- new net GFO3: C37.1, R58.2, U6.7 (IN3)
- new net SCLK: U5.16 (SCLK), U6.16 (SCLK), U7.16 (SCLK)
- new net STemp10: C27.1, R41.2, U7.5 (IN1)
- new net STemp11: C28.1, R42.2, U7.6 (IN2)
- new net STemp2: C19.1, R26.2, U5.5 (IN1)
- new net STemp3: C20.1, R27.2, U5.6 (IN2)
- new net STemp4: C21.1, R28.2, U5.7 (IN3)
- new net STemp5: C22.1, R29.2, U5.8 (IN4)
- new net STemp6: C23.1, R30.2, U5.9 (IN5)
- new net STemp7: C24.1, R31.2, U5.10 (IN6)
- new net STemp8: C25.1, R39.2, U5.11 (IN7)
- new net STemp9: C26.1, R40.2, U7.4 (IN0)
- new net nCS_1: U5.1 (~CS)
- new net nCS_2: U7.1 (~CS)
- new net nCS_3: U6.1 (~CS)
Other:
- note added: "Check Ground Fault Sensors\n"
- moved on the sheet: C18, J1, R25

Commit message: Schematic Clean up, Fan Actuation, SSR actuation sch fix
Parts:
- C24: renamed from C18; footprint (none) -> Capacitor_SMD:C_0603_1608Metric_Pad1.08x0.95mm_HandSolder
- C25: renamed from C19; footprint (none) -> Capacitor_SMD:C_0603_1608Metric_Pad1.08x0.95mm_HandSolder
- C26: renamed from C20; footprint (none) -> Capacitor_SMD:C_0603_1608Metric_Pad1.08x0.95mm_HandSolder
- C27: renamed from C21; footprint (none) -> Capacitor_SMD:C_0603_1608Metric_Pad1.08x0.95mm_HandSolder
- C28: renamed from C22; footprint (none) -> Capacitor_SMD:C_0603_1608Metric_Pad1.08x0.95mm_HandSolder
- C29: renamed from C23; footprint (none) -> Capacitor_SMD:C_0603_1608Metric_Pad1.08x0.95mm_HandSolder
- C30: renamed from C24; footprint (none) -> Capacitor_SMD:C_0603_1608Metric_Pad1.08x0.95mm_HandSolder
- C31: renamed from C25; footprint (none) -> Capacitor_SMD:C_0603_1608Metric_Pad1.08x0.95mm_HandSolder
- C32: renamed from C26; footprint (none) -> Capacitor_SMD:C_0603_1608Metric_Pad1.08x0.95mm_HandSolder
- C33: renamed from C27; footprint (none) -> Capacitor_SMD:C_0603_1608Metric_Pad1.08x0.95mm_HandSolder
- C34: renamed from C28; footprint (none) -> Capacitor_SMD:C_0603_1608Metric_Pad1.08x0.95mm_HandSolder
- C35: renamed from C29; footprint (none) -> Capacitor_SMD:C_0603_1608Metric_Pad1.08x0.95mm_HandSolder
- C36: renamed from C30; footprint (none) -> Capacitor_SMD:C_0603_1608Metric_Pad1.08x0.95mm_HandSolder
- C37: renamed from C31; footprint (none) -> Capacitor_SMD:C_0603_1608Metric_Pad1.08x0.95mm_HandSolder
- C38: renamed from C32; footprint (none) -> Capacitor_SMD:C_0603_1608Metric_Pad1.08x0.95mm_HandSolder
- C39: renamed from C33; footprint (none) -> Capacitor_SMD:C_0603_1608Metric_Pad1.08x0.95mm_HandSolder
- C40: renamed from C34; footprint (none) -> Capacitor_SMD:C_0603_1608Metric_Pad1.08x0.95mm_HandSolder
- C41: renamed from C35; footprint (none) -> Capacitor_SMD:C_0603_1608Metric_Pad1.08x0.95mm_HandSolder
- C42: renamed from C36; footprint (none) -> Capacitor_SMD:C_0603_1608Metric_Pad1.08x0.95mm_HandSolder
- C43: renamed from C37; footprint (none) -> Capacitor_SMD:C_0603_1608Metric_Pad1.08x0.95mm_HandSolder
- C44: renamed from C38; footprint (none) -> Capacitor_SMD:C_0603_1608Metric_Pad1.08x0.95mm_HandSolder
- C45: renamed from C39; footprint (none) -> Capacitor_SMD:C_0603_1608Metric_Pad1.08x0.95mm_HandSolder
- C46: renamed from C40; footprint (none) -> Capacitor_SMD:C_0603_1608Metric_Pad1.08x0.95mm_HandSolder
- C47: renamed from C41; footprint (none) -> Capacitor_SMD:C_0603_1608Metric_Pad1.08x0.95mm_HandSolder
- C48: renamed from C42; footprint (none) -> Capacitor_SMD:C_0603_1608Metric_Pad1.08x0.95mm_HandSolder
- C49: renamed from C43; footprint (none) -> Capacitor_SMD:C_0603_1608Metric_Pad1.08x0.95mm_HandSolder
- C50: renamed from C44; footprint (none) -> Capacitor_SMD:C_0603_1608Metric_Pad1.08x0.95mm_HandSolder
- C51: renamed from C45; footprint (none) -> Capacitor_SMD:C_0603_1608Metric_Pad1.08x0.95mm_HandSolder
- C52: renamed from C46; footprint (none) -> Capacitor_SMD:C_0603_1608Metric_Pad1.08x0.95mm_HandSolder
- C53: renamed from C47; footprint (none) -> Capacitor_SMD:C_0603_1608Metric_Pad1.08x0.95mm_HandSolder
- C54: renamed from C48; footprint (none) -> Capacitor_SMD:C_0603_1608Metric_Pad1.08x0.95mm_HandSolder
- C55: renamed from C49; footprint (none) -> Capacitor_SMD:C_0603_1608Metric_Pad1.08x0.95mm_HandSolder
- C56: renamed from C50; footprint (none) -> Capacitor_SMD:C_0603_1608Metric_Pad1.08x0.95mm_HandSolder
- C57: renamed from C51; footprint (none) -> Capacitor_SMD:C_0603_1608Metric_Pad1.08x0.95mm_HandSolder
- C58: renamed from C52; footprint (none) -> Capacitor_SMD:C_0603_1608Metric_Pad1.08x0.95mm_HandSolder
- C59: renamed from C53; footprint (none) -> Capacitor_SMD:C_0603_1608Metric_Pad1.08x0.95mm_HandSolder
- C60: renamed from C54; footprint (none) -> Capacitor_SMD:C_0603_1608Metric_Pad1.08x0.95mm_HandSolder
- C61: renamed from C55; footprint (none) -> Capacitor_SMD:C_0603_1608Metric_Pad1.08x0.95mm_HandSolder
- J11: renamed from J1; footprint (none) -> Connector_Molex:Molex_MicroClasp_55935-0310_1x03_P2.00mm_Horizontal
- J12: renamed from J2; footprint (none) -> Connector_Molex:Molex_MicroClasp_55935-0310_1x03_P2.00mm_Horizontal
- J13: renamed from J3; footprint (none) -> Connector_Molex:Molex_MicroClasp_55935-0310_1x03_P2.00mm_Horizontal
- J14: renamed from J4; footprint (none) -> Connector_Molex:Molex_MicroClasp_55935-0310_1x03_P2.00mm_Horizontal
- J15: renamed from J5; footprint (none) -> Connector_Molex:Molex_MicroClasp_55935-0310_1x03_P2.00mm_Horizontal
- J16: renamed from J6; footprint (none) -> Connector_Molex:Molex_MicroClasp_55935-0310_1x03_P2.00mm_Horizontal
- J17: renamed from J7; footprint (none) -> Connector_Molex:Molex_MicroClasp_55935-0310_1x03_P2.00mm_Horizontal
- J18: renamed from J8; footprint (none) -> Connector_Molex:Molex_Micro-Latch_53254-0470_1x04_P2.00mm_Horizontal
- J19: renamed from J9; footprint (none) -> Connector_Molex:Molex_Micro-Latch_53254-0470_1x04_P2.00mm_Horizontal
- J20: renamed from J10; footprint (none) -> Connector_Molex:Molex_Micro-Latch_53254-0470_1x04_P2.00mm_Horizontal
- J21: renamed from J11; footprint (none) -> Connector_Molex:Molex_Micro-Fit_3.0_43045-0210_2x01-1MP_P3.00mm_Horizontal
- J22: renamed from J12; footprint (none) -> Connector_Molex:Molex_MicroClasp_55935-0310_1x03_P2.00mm_Horizontal
- J23: renamed from J13; footprint (none) -> Connector_Molex:Molex_MicroClasp_55935-0310_1x03_P2.00mm_Horizontal
- J24: renamed from J14; footprint (none) -> Connector_Molex:Molex_MicroClasp_55935-0310_1x03_P2.00mm_Horizontal
- J25: renamed from J15; footprint (none) -> Connector_Molex:Molex_Nano-Fit_105313-xx08_1x08_P2.50mm_Horizontal
- J26: renamed from J16; footprint (none) -> Connector_Molex:Molex_Micro-Fit_3.0_43650-0400_1x04_P3.00mm_Horizontal
- J27: renamed from J17; footprint (none) -> Connector_Molex:Molex_Micro-Fit_3.0_43650-0400_1x04_P3.00mm_Horizontal
- J28: renamed from J18; footprint (none) -> Connector_Molex:Molex_Micro-Fit_3.0_43650-0400_1x04_P3.00mm_Horizontal
- J29: renamed from J19; footprint (none) -> Connector_Molex:Molex_Micro-Fit_3.0_43650-0400_1x04_P3.00mm_Horizontal
- J30: renamed from J20; footprint (none) -> Connector_Molex:Molex_MicroClasp_55935-0610_1x06_P2.00mm_Horizontal
- J31: renamed from J21; footprint (none) -> Connector_Molex:Molex_Micro-Fit_3.0_43650-0400_1x04_P3.00mm_Horizontal
- J32: renamed from J22; footprint (none) -> Connector_Molex:Molex_Micro-Fit_3.0_43650-0400_1x04_P3.00mm_Horizontal
- R18, R19, R20, R21, R22, R23, R24, R25, R26, R27, R28, R29, R30, R31, R32, R33, R34, R35, R36, R37, R38, R39, R40, R41, R42, R43, R44, R45, R46, R47, R48, R49, R50, R51, R52, R53, R54, R55, R56, R57, R58, R59, R60, R61, R62, R63, R64, R65, R66, R67, R68, R69: footprint (none) -> Resistor_SMD:R_0603_1608Metric_Pad0.98x0.95mm_HandSolder
- U5, U6, U7: footprint SOP65P640X120-16N -> boringlib-master:SOP65P640X120-16N; symbol ADC128S022CIMT:ADC128S022CIMT -> LokiV1-rescue:ADC128S022CIMT-ADC128S022CIMT
