File: PCB_PLV008_Loki/AvionicsHeartBeatTemplate.sch (KiCad schematic (older format))
At the start: 0 parts

Commit message: Schematic Clean up, Fan Actuation, SSR actuation sch fix
Parts:
- added C62, C63, C64, C65, C66, C67: 0.1uF, Capacitor_SMD:C_0603_1608Metric_Pad1.05x0.95mm_HandSolder, symbol Device:C
- added C68: 1uF, Capacitor_SMD:C_0603_1608Metric_Pad1.05x0.95mm_HandSolder, symbol Device:C
- added D8: GREEN, LED_SMD:LED_0805_2012Metric_Pad1.15x1.40mm_HandSolder, symbol Device:LED
- added D9: BLUE, LED_SMD:LED_0805_2012Metric_Pad1.15x1.40mm_HandSolder, symbol Device:LED
- added Q5: DMG2302UK-7, Package_TO_SOT_SMD:SOT-23_Handsoldering, symbol Device:Q_NMOS_GDS
- added Q6: DMP2123L-7, Package_TO_SOT_SMD:SOT-23_Handsoldering, symbol Device:Q_PMOS_GDS
- added R70, R71, R73, R74, R76, R77: DNP, Resistor_SMD:R_0603_1608Metric_Pad1.05x0.95mm_HandSolder, symbol Device:R_US
- added R72, R75: DNP, Resistor_SMD:R_0201_0603Metric_Pad0.64x0.40mm_HandSolder, symbol Device:R_US
- added R78, R84: 47K, Resistor_SMD:R_0603_1608Metric_Pad1.05x0.95mm_HandSolder, symbol Device:R_US
- added R79: 1K, Resistor_SMD:R_0201_0603Metric_Pad0.64x0.40mm_HandSolder, symbol Device:R_US
- added R80: 1M, Resistor_SMD:R_0201_0603Metric_Pad0.64x0.40mm_HandSolder, symbol Device:R_US
- added R81: 280K, Resistor_SMD:R_0201_0603Metric_Pad0.64x0.40mm_HandSolder, symbol Device:R_US
- added R82: 604K, Resistor_SMD:R_0201_0603Metric_Pad0.64x0.40mm_HandSolder, symbol Device:R_US
- added R83: 47K, Resistor_SMD:R_0201_0603Metric_Pad0.64x0.40mm_HandSolder, symbol Device:R_US
- added R85: 1K, Resistor_SMD:R_0603_1608Metric_Pad1.05x0.95mm_HandSolder, symbol Device:R_US
- added U10, U16: 74HC08, Package_SO:SOIC-14_3.9x8.7mm_P1.27mm, symbol LokiV1-rescue:74HC08-boringlib
- added U11, U8: 74HC21, Package_SO:SOIC-14_3.9x8.7mm_P1.27mm, symbol LokiV1-rescue:74HC21-boringlib
- added U12, U13, U14, U9: 74HC266, Package_SO:SOIC-14_3.9x8.7mm_P1.27mm, symbol LokiV1-rescue:74HC266-boringlib
- added U15: 74LVC1G17, Package_TO_SOT_SMD:SOT-23-5_HandSoldering, symbol LokiV1-rescue:74LVC1G17-boringlib
- added U17: LTC6993xS6-1, Package_TO_SOT_SMD:TSOT-23-6, symbol Timer:LTC6993xS6-1
Connections:
- new net: U10.1, U8.6
- new net: U10.2, U8.8
- new net: R70.2, R74.2, U9.2
- new net: U11.1, U9.3
- new net: R71.2, R75.2, U12.2
- new net: U11.2, U12.3
- new net: R72.2, R76.2, U13.2
- new net: U11.4, U13.3
- new net: R73.2, R77.2, U14.2
- new net: U11.5, U14.3
- new net: D8.2 (A), U10.3, U16.1
- new net: U11.6, U16.2
- new net: U16.3, U17.1 (TRIG)
- new net: R82.1, U17.3 (SET)
- new net: R80.2, R81.1, U17.4 (DIV)
- new net: Q5.1 (G), U17.6 (OUT)
- new net: Q5.2 (D), Q6.1 (G), R83.2
- new net: D8.1 (K), R79.1
- new net: D9.1 (K), R85.1
- new net +5V: C62.1, C63.1, C64.1, C65.1, C66.1, C67.1, C68.1, Q6.3 (S), R74.1, R75.1, R76.1, R77.1, R80.1, R83.1, U10.14 (VCC), U11.14 (VCC), U15.5 (VCC), U17.5 (V+), U8.14 (VCC), U9.14 (VCC)
- new net GND: C62.2, C63.2, C64.2, C65.2, C66.2, C67.2, C68.2, Q5.3 (S), R70.1, R71.1, R72.1, R73.1, R79.2, R81.2, R82.2, R84.2, R85.2, U10.7 (GND), U11.7 (GND), U15.3 (GND), U17.2 (GND), U8.7 (GND), U9.7 (GND)
- new net HEARTBEAT: Q6.2 (D), R78.2, R84.1, U15.2
- new net HEARTBEAT_ADDRESS_1: U9.1
- new net HEARTBEAT_ADDRESS_2: U12.1
- new net HEARTBEAT_ADDRESS_3: U13.1
- new net HEARTBEAT_ADDRESS_4: U14.1
- new net HEARTBEAT_BUFF: D9.2 (A), U15.4
- new net HEARTBEAT_INPUT_1: U8.1
- new net HEARTBEAT_INPUT_2: U8.2
- new net HEARTBEAT_INPUT_3: U8.4
- new net HEARTBEAT_INPUT_4: U8.5
- new net HEARTBEAT_INPUT_5: U8.9
- new net HEARTBEAT_INPUT_6: U8.10
- new net HEARTBEAT_INPUT_7: U8.12
- new net HEARTBEAT_RESTART: R78.1, U8.13
Other:
- note added: "6.25ms timer\nw/ 16 addresses\nthis gives 10Hz cycle"
- note added: "Use stuffing options to select\nboard heartbeat address"
