File: PCB_PLV008_Loki/AvionicsHeartbeat.sch (KiCad schematic (older format))
At the start: 33 parts, among them Q1 DMG2302UK-7, Q2 DMP2123L-7, U1 74HC21, U2 74HC266, U3 74HC08, U4 74HC21, U5 74LVC1G17, U6 LTC6993xS6-1

Commit message: Add files via upload
Parts:
- renumbered C1 to C11, C2 to C12, C3 to C13, C4 to C14, C5 to C15, C6 to C16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

Commit message: Schematic Clean up, Fan Actuation, SSR actuation sch fix
Parts:
- gave numbers to parts that had none: 5
- renumbered C11 to C1, C12 to C2, C13 to C3, C14 to C4, C15 to C5, C16 to C6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
