File: PCB_PLV008_Loki/LV_PowerConversion.sch (KiCad schematic (older format))
At the start: 23 parts

Commit message: Add files via upload
Parts:
- removed C?: C, symbol Device:C
- removed F? (x2): Fuse, symbol Device:Fuse
- removed FL?: FN405-10-02, Filter:Filter_Schaffner_FN405, symbol Filter:FN405-10-02
- removed J?: Conn_01x02, symbol Connector_Generic:Conn_01x02
- added C59, C66: C, symbol Device:C
- added C62, C65: 470uF, symbol Device:CP
- added C63, C64: 2.2uF, symbol Device:C
- added C67: C11, symbol Device:C
- added D3: 5KPxxA, Diode_THT:D_P600_R-6_P20.00mm_Horizontal, symbol Diode:5KPxxA
- added FL2: FN405-10-02, Filter:Filter_Schaffner_FN405, symbol Filter:FN405-10-02
- added J23, J26: Conn_01x02, symbol Connector_Generic:Conn_01x02
- added PS1: TUNS700F28, TUNS700F28, symbol TUNS700F28:TUNS700F28
- added TH2: Thermistor_NTC_US, symbol Device:Thermistor_NTC_US
- gave numbers to parts that had none: 18
Connections:
- net GND: now also C59.2, C62.1, C62.2, C63.1, C63.2, C66.2, D3.2 (A2), FL2.3 (E), J26.1 (Pin_1), J26.2 (Pin_2), PS1.3 (-VOUT), PS1.4 (+VOUT), PS1.5 (-S), PS1.6 (+S)
- net at C56.1, FL1.5 (P), RV1.1: now also J23.1 (Pin_1)
- net at C56.2, FL1.1 (N), RV1.2: now also J23.2 (Pin_2)
- net at C57.2, C58.1, FL1.2 (N'): now also FL2.1 (N)
- net at C57.1, FL1.4 (P'): now also C59.1, FL2.5 (P)
- net at C60.1, C61.1, R70.1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: now also FL2.4 (P'), PS1.1 (AC2); no longer C60.2, C61.2, R72.2, R75.2, RV2.1
- net at RV2.2: now also RV3.2, D3.1 (A1)
- net at TH1.1: now also J24.1 (Pin_1)
- new net: C60.2, C61.2, FL2.2 (N'), PS1.2 (AC1), R72.2, R75.2, RV2.1
- new net: C64.2, C65.2, C66.1, C67.1, PS1.11 (-BC), TH2.2
- new net: C65.1, C67.2, PS1.12 (+BC), TH2.1
- new net: C64.1, PS1.13 (R)
- new net VTrim: PS1.7 (TRM)
Other:
- moved on the sheet: C56, C57, C58, C60, C61, FL1, J24, J25, R70, R71, R72, R73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

Commit message: Add files via upload
Parts:
- C56, C57, C60, C61: value C -> 1.5uF
- C58, C59, C66: value C -> 2200pF
- R70, R71, R72, R73, R74, R75: value R_US -> 68K
- RV1, RV2, RV3: value Varistor_US -> 620V
- renumbered C67 to C0.68uF
Other:
- moved on the sheet: C0.68uF, C56, C57, C58, C59, C60, C61, C62, C63, C64, C65, C66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

Commit message: Schematic Clean up, Fan Actuation, SSR actuation sch fix
Parts:
- C0.68uF1: renamed from C0.68uF; footprint (none) -> Capacitor_SMD:C_0603_1608Metric_Pad1.08x0.95mm_HandSolder
- C11: renamed from C56; footprint (none) -> Capacitor_SMD:C_0603_1608Metric_Pad1.08x0.95mm_HandSolder
- C12: renamed from C57; footprint (none) -> Capacitor_SMD:C_0603_1608Metric_Pad1.08x0.95mm_HandSolder
- C13: renamed from C58; footprint (none) -> Capacitor_SMD:C_0603_1608Metric_Pad1.08x0.95mm_HandSolder
- C14: renamed from C59; footprint (none) -> Capacitor_SMD:C_0603_1608Metric_Pad1.08x0.95mm_HandSolder
- C15: renamed from C60; footprint (none) -> Capacitor_SMD:C_0603_1608Metric_Pad1.08x0.95mm_HandSolder
- C16: renamed from C61; footprint (none) -> Capacitor_SMD:C_0603_1608Metric_Pad1.08x0.95mm_HandSolder
- C17: renamed from C62; footprint (none) -> Capacitor_THT:CP_Radial_D18.0mm_P7.50mm
- C18: renamed from C63; footprint (none) -> Capacitor_SMD:C_0603_1608Metric_Pad1.08x0.95mm_HandSolder
- C19: renamed from C64; footprint (none) -> Capacitor_SMD:C_0603_1608Metric_Pad1.08x0.95mm_HandSolder
- C20: renamed from C65; footprint (none) -> Capacitor_SMD:C_1210_3225Metric_Pad1.33x2.70mm_HandSolder
- C21: renamed from C66; footprint (none) -> Capacitor_SMD:C_0603_1608Metric_Pad1.08x0.95mm_HandSolder
- J2: renamed from J23; footprint (none) -> Connector_Molex:Molex_Micro-Fit_3.0_43650-0200_1x02_P3.00mm_Horizontal
- J3: renamed from J24; footprint (none) -> Connector_Molex:Molex_Micro-Fit_3.0_43650-0200_1x02_P3.00mm_Horizontal
- J4: renamed from J25; footprint (none) -> Connector_Molex:Molex_Micro-Fit_3.0_43650-0200_1x02_P3.00mm_Horizontal
- J5: renamed from J26; footprint (none) -> Connector_Molex:Molex_Micro-Fit_3.0_43650-0200_1x02_P3.00mm_Horizontal
- PS1: footprint TUNS700F28 -> TUNS700F28:TUNS700F28; symbol TUNS700F28:TUNS700F28 -> LokiV1-rescue:TUNS700F28-TUNS700F28
- R10: renamed from R72; footprint (none) -> Resistor_SMD:R_0603_1608Metric_Pad0.98x0.95mm_HandSolder
- R11: renamed from R73; footprint (none) -> Resistor_SMD:R_0603_1608Metric_Pad0.98x0.95mm_HandSolder
- R12: renamed from R74; footprint (none) -> Resistor_SMD:R_0603_1608Metric_Pad0.98x0.95mm_HandSolder
- R13: renamed from R75; footprint (none) -> Resistor_SMD:R_0603_1608Metric_Pad0.98x0.95mm_HandSolder
- R8: renamed from R70; footprint (none) -> Resistor_SMD:R_0603_1608Metric_Pad0.98x0.95mm_HandSolder
- R9: renamed from R71; footprint (none) -> Resistor_SMD:R_0603_1608Metric_Pad0.98x0.95mm_HandSolder
- RV1, RV2, RV3: footprint (none) -> Resistor_THT:R_Axial_DIN0614_L14.3mm_D5.7mm_P5.08mm_Vertical
- TH1: value Thermistor_NTC -> 120; footprint (none) -> Resistor_THT:R_Axial_DIN0614_L14.3mm_D5.7mm_P5.08mm_Vertical
- TH2: value Thermistor_NTC_US -> 120; footprint (none) -> Resistor_THT:R_Axial_DIN0614_L14.3mm_D5.7mm_P5.08mm_Vertical
- renumbered D3 to D2
Other:
- moved on the sheet: J3, J4
