File: PCB_PLV008_Loki/LokiV1.sch (KiCad schematic (older format))
At the start: 23 parts

Commit message: Add files via upload
Parts:
- removed D? (x3): 1N53xxB, Diode_THT:D_DO-201_P15.24mm_Horizontal, symbol Diode:1N53xxB
- removed J? (x3): Conn_01x02, symbol Connector_Generic:Conn_01x02
- removed Q? (x3): DMG2302U, Package_TO_SOT_SMD:SOT-23, symbol Transistor_FET:DMG2302U
- removed R? (x3): R_Small, symbol Device:R_Small
- added C10: 0.1uF, symbol Device:C
- added C8, C9: C, symbol Device:C
- added D?: D_Schottky, symbol Device:D_Schottky
- added F?: Fuse, symbol Device:Fuse
- added J?: Conn_01x12, symbol Connector_Generic:Conn_01x12
- added JP1: Jumper_NC_Small, symbol Device:Jumper_NC_Small
- added R1: R_US, symbol Device:R_US
- added U2: BME280, Package_LGA:Bosch_LGA-8_2.5x2.5mm_P0.65mm_ClockwisePinNumbering, symbol Sensor:BME280
- gave numbers to parts that had none: 11
Connections:
- net +24V: now also D?.1 (K)
- net +3V3: now also C10.1, C8.2, C9.1, U2.6 (VDDIO), U2.8 (VDD)
- net GND: now also C10.2, C8.1, C9.2, J?.11 (Pin_11), J?.12 (Pin_12), U2.1 (GND), U2.7 (GND)
- net at U3.6 (CANL): now also JP1.2
- net at U3.7 (CANH): now also R1.1
- net ControlLaptop_Relay: no longer names the net of NCLO1.65 (PB4/SPI1_MISO/PWM3_1)
- new net: JP1.1, R1.2
- new net: D?.2 (A), F?.2
- new net CANH: J?.7 (Pin_7)
- new net CANL: J?.8 (Pin_8)
- new net CSB: U2.2 (CSB)
- new net HeartBeat: J?.2 (Pin_2)
- new net HeartBeat_Address_1: J?.6 (Pin_6)
- new net HeartBeat_Address_2: J?.5 (Pin_5)
- new net HeartBeat_Address_3: J?.4 (Pin_4)
- new net HeartBeat_Address_4: J?.3 (Pin_3)
- new net SPI_DIN: U2.3 (SDI)
- new net SPI_DOUT: U2.5 (SDO)
- new net SPI_SCLK: U2.4 (SCK)
- new net VIN: F?.1, J?.10 (Pin_10), J?.9 (Pin_9)
- no-connect marks 0 -> 1
Other:
- moved on the sheet: C1, C2, C3, C4, C5, C6, C7, FB1, U1, U3

Commit message: Add files via upload
Parts:
- added R?: 0, symbol Device:R_US
Connections:
- net +5V: now also R?.1
- net AvionicsHeartBeatTemplate/HeartBeat_Input_1: now also R?.2
- net CANH: now also J?.6 (Pin_6); no longer J?.7 (Pin_7)
- net CANL: now also J?.5 (Pin_5); no longer J?.8 (Pin_8)
- net GND: now also J?.1 (Pin_1), J?.2 (Pin_2); no longer J?.11 (Pin_11), J?.12 (Pin_12)
- net HeartBeat: now also J?.11 (Pin_11); no longer J?.2 (Pin_2)
- net HeartBeat_Address_1: now also J?.7 (Pin_7); no longer J?.6 (Pin_6)
- net HeartBeat_Address_2: now also J?.8 (Pin_8); no longer J?.5 (Pin_5)
- net HeartBeat_Address_3: now also J?.9 (Pin_9); no longer J?.4 (Pin_4)
- net HeartBeat_Address_4: now also J?.10 (Pin_10); no longer J?.3 (Pin_3)
- net VIN: now also J?.3 (Pin_3), J?.4 (Pin_4); no longer J?.10 (Pin_10), J?.9 (Pin_9)
- no-connect marks 1 -> 7
Other:
- moved on the sheet: C1, C2, C3, C4, C5, C6, C7, D?, F?, FB1, J?, U1

Commit message: Schematic Clean up, Fan Actuation, SSR actuation sch fix
Parts:
- removed R?: 0, symbol Device:R_US
- added R1, R2, R3, R4, R5, R6: 0, Resistor_SMD:R_0603_1608Metric_Pad0.98x0.95mm_HandSolder, symbol Device:R_US
- C1: footprint (none) -> Capacitor_SMD:C_1210_3225Metric_Pad1.33x2.70mm_HandSolder
- C10: footprint (none) -> Capacitor_SMD:C_0603_1608Metric_Pad1.08x0.95mm_HandSolder
- C2: renamed from C4; footprint (none) -> Capacitor_SMD:C_1210_3225Metric_Pad1.33x2.70mm_HandSolder
- C3: renamed from C5; footprint (none) -> Capacitor_SMD:C_0603_1608Metric_Pad1.08x0.95mm_HandSolder
- C4: renamed from C6; footprint (none) -> Capacitor_SMD:C_0603_1608Metric_Pad1.08x0.95mm_HandSolder
- C5: renamed from C7; footprint (none) -> Capacitor_SMD:C_0603_1608Metric_Pad1.08x0.95mm_HandSolder
- C6: renamed from C2; footprint (none) -> Capacitor_SMD:C_1210_3225Metric_Pad1.33x2.70mm_HandSolder
- C7: renamed from C3; footprint (none) -> Capacitor_SMD:C_0603_1608Metric_Pad1.08x0.95mm_HandSolder
- C8, C9: value C -> 100nF; footprint (none) -> Capacitor_SMD:C_0603_1608Metric_Pad1.08x0.95mm_HandSolder
- D1: renamed from D?; footprint (none) -> BoringFootprints:DO-221AC
- F1: renamed from F?; footprint (none) -> BoringFootprints:BelFuse_0679H
- FB1: footprint (none) -> Inductor_SMD:L_0201_0603Metric_Pad0.64x0.40mm_HandSolder
- J1: renamed from J?; footprint (none) -> Connector_Molex:Molex_Micro-Fit_3.0_43045-1200_2x06_P3.00mm_Horizontal
- JP1: footprint (none) -> Jumper:SolderJumper-2_P1.3mm_Bridged_RoundedPad1.0x1.5mm
- NCLO1: symbol boringlib:NUCLEO-L476RG -> LokiV1-rescue:NUCLEO-L476RG-boringlib
- R7: renamed from R1; value R_US -> 120; footprint (none) -> Resistor_SMD:R_0603_1608Metric_Pad0.98x0.95mm_HandSolder
- U1: symbol boringlib:R-78B-2.0 -> LokiV1-rescue:R-78B-2.0-boringlib
Connections:
- net SPI_DOUT is gone; now on net SPI_MOSI: U2.5 (SDO)
- net +5V: now also R1.1, R2.1, R3.1, R4.1, R5.1, R6.1
- net ACVO1: now also NCLO1.38 (PC0/ADC/I2C3_SCL/UART1_RX)
- net ACVO2: now also NCLO1.36 (PC1/ADC/I2C3_SDA/UART1_TX)
- net ADC_nCS_1: now also NCLO1.63 (PB10/I2C2_SCL/SPI2_SCLK/UART1_RX/UART3_TX/PWM2_3)
- net ADC_nCS_2: now also NCLO1.56 (PB11/I2C2_SDA/UART3_RX/UART1_TX/PWM2_4)
- net ADC_nCS_3: now also NCLO1.54 (PB12/SPI2_SSEL)
- net AvionicsHeartBeatTemplate/HeartBeat_Input_1: now also R1.2
- net CSB: now also NCLO1.43 (PB9/SPI2_SSEL/CAN1_TD/I2C1_SDA/PWM4_4)
- net ControlLaptopLine_Relay: now also NCLO1.72 (PC4/ADC/UART3_TX)
- net HeartBeat_Input_7: now also NCLO1.62 (PB1/ADC/PWM3_4)
- net HeartBeat_Restart: now also NCLO1.60 (PB2)
- net InputLine_Bleeder: now also NCLO1.44 (PC5/ADC/UART3_RX)
- net InputLine_Relay: now also NCLO1.37 (PC3/ADC/SPI2_MOSI)
- net LowVoltageLine_Relay: now also NCLO1.35 (PC2/ADC/SPI2_MISO)
- net SPI_SCLK: now also NCLO1.68 (PB13/I2C2_SCL/SPI2_SCLK/PWM1_1N)
- net VTrim: now also NCLO1.34 (PB0/ADC/PWM3_3)
- net HeartBeat_Buff: now reaches NCLO1.13 (PA13)
- net SPI_MOSI: now reaches NCLO1.64 (PB15/SPI2_MOSI/PWM1_3N)
- net SPI_MSIO: now reaches NCLO1.66 (PB14/I2C2_SDA/SPI2_MISO/PWM1_2N)
- net SPI_DIN renamed SPI_MISO
- new net AvionicsHeartBeatTemplate/HeartBeat_Input_2: R2.2
- new net AvionicsHeartBeatTemplate/HeartBeat_Input_3: R3.2
- new net AvionicsHeartBeatTemplate/HeartBeat_Input_4: R4.2
- new net AvionicsHeartBeatTemplate/HeartBeat_Input_5: R5.2
- new net AvionicsHeartBeatTemplate/HeartBeat_Input_6: R6.2
- no-connect marks 7 -> 39
Other:
- moved on the sheet: C1, C10, C2, C3, C4, C5, C6, C7, C8, C9, D1, F1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
